File: mec1723.kicad_sch (KiCad schematic)
At the start: 53 parts, among them SW3001 SW_B3U-1000P_SMD, SW3002 SW_B3U-1000P_SMD, U3001 MEC1723N-B0-I/SZ, Y3001 Resonator_32.768kHz_ECX-31B

Commit message: [#103224] Add crucial signals, add strapping
Parts:
- added C3018: C_1u_6.3V_X6S_0402, antmicro-footprints:C_0402_1005Metric, symbol Antmicro Symbols:C_1u_6.3V_X6S_0402
- added R3026, R3029, R3030, R3031, R3032: R_10k_0402, antmicro-footprints:R_0402_1005Metric, symbol Antmicro Symbols:R_10k_0402
- added R3027: R_100R_0402, antmicro-footprints:R_0402_1005Metric, symbol Antmicro Symbols:R_100R_0402
- added R3028: R_0R_0402, antmicro-footprints:R_0402_1005Metric, symbol Antmicro Symbols:R_0R_0402
- added SW3003: SW_B3U-1000P_SMD, antmicro-footprints:SW_B3U-1000P_SMD, symbol Antmicro Symbols:SW_B3U-1000P_SMD
Connections:
- net +3V3: now also R3026.1, R3030.2, R3031.2
- net CR_STRAP: now also R3031.1, R3032.2
- net GND: now also U3001.H11 (GPIO044/VREF_VTT), C3018.1, R3029.1, SW3003.2
- net JTAG_STRAP: now also R3029.2, R3030.1
- net PWRGD_S0iX: now reaches U3001.F2 (GPIO226/PWRGD_S0iX/CMP_VREF0)
- net PWRGD_S0iX: now also R3028.1
- new net: R3027.2, SW3003.1
- new net: C3018.2, R3026.2, R3027.1, R3028.2
- no-connect marks 3 -> 2
Other:
- note removed: "PECI Vref"
- moved on the sheet: C3002, C3003, Y3001
