File: power.kicad_sch (KiCad schematic)
At the start: 0 parts

Commit message: [#103224] Add power section schematic
Parts:
- added C4001: C_10u_16V_0603, antmicro-footprints:C_0603_1608Metric, symbol antmicroCapacitors0603:C_10u_16V_0603
- added C4002: C_100n_50V_X8L_0402, antmicro-footprints:C_0402_1005Metric, symbol antmicroCapacitors0402:C_100n_50V_X8L_0402
- added C4003: C_22u_16V_0603, antmicro-footprints:C_0603_1608Metric_EIA, symbol antmicroCapacitors0603:C_22u_16V_0603
- added C4004: C_22u_0603, antmicro-footprints:C_0603_1608Metric, symbol antmicroCapacitors0603:C_22u_0603
- added C4005, C4006: C_10u_10V_0402, antmicro-footprints:C_0402_1005Metric, symbol antmicroCapacitors0402:C_10u_10V_0402
- added D4001, D4003, D4004: LED_G_0603_LTST-C190GKT, antmicro-footprints:LED_0603_1608Metric_G, symbol antmicroLEDIndicationDiscrete:LED_G_0603_LTST-C190GKT
- added L4001: L_3u3_6.6A_XEL4030, antmicro-footprints:L_Coilcraft-XEL4030, symbol antmicroFixedInductors:L_3u3_6.6A_XEL4030
- added Q4001: DMG1012T-7, antmicro-footprints:SOT-523, symbol antmicroTransistorsFETsMOSFETsSingle:DMG1012T-7
- added R4001, R4004, R4005, R4009, R4017, R4018: R_10k_0402, antmicro-footprints:R_0402_1005Metric, symbol antmicroResistors0402:R_10k_0402
- added R4002, R4006: R_1k_0402, antmicro-footprints:R_0402_1005Metric, symbol Antmicro Symbols:R_1k_0402
- added R4003, R4015, R4016: R_0R_0402, antmicro-footprints:R_0402_1005Metric, symbol antmicroResistors0402:R_0R_0402
- added R4007: R_31k6_0402, antmicro-footprints:R_0402_1005Metric, symbol antmicroResistors0402:R_31k6_0402
- added R4011: R_0R_22.4A_0603, antmicro-footprints:R_0603_1608Metric, symbol antmicroResistors0603:R_0R_22.4A_0603
- added R4012, R4013: R_100k_0402, antmicro-footprints:R_0402_1005Metric, symbol antmicroResistors0402:R_100k_0402
- added R4014: R_160k_0402, antmicro-footprints:R_0402_1005Metric, symbol antmicroResistors0402:R_160k_0402
- added TP4001, TP4002: TP_0.75mm_SMD, antmicro-footprints:TP_SMD_0.75mm, symbol antmicroTestPoints:TP_0.75mm_SMD
- added U4001: AP62301_TSOT, antmicro-footprints:TSOT23-6, symbol antmicroDCDCConverters:AP62301_TSOT
- added U4002: TLV76701_WSON, antmicro-footprints:WSON-6-1EP_2x2mm_P0.65mm, symbol antmicroPMICVoltageRegulatorsLinear:TLV76701_WSON
Connections:
- new net: D4004.1 (C), Q4001.3 (D)
- new net: D4004.2 (A), R4006.1
- new net: D4003.2 (A), R4002.1
- new net: D4001.2 (A), R4001.1
- new net: R4016.2, R4017.1, R4018.2, U4002.4 (EN)
- new net: R4012.1, R4013.2
- new net +1V8: Q4001.1 (G), R4015.2, TP4002.1
- new net +3V3: C4005.2, R4002.2, R4006.2, R4011.2, R4017.2, TP4001.1, U4002.6 (IN)
- new net 1V8_FB: R4013.1, R4014.2, U4002.2 (FB)
- new net 1V8_R: C4006.2, R4012.2, R4015.1, U4002.1 (OUT)
- new net 3V3_OUT: C4003.2, C4004.2, L4001.2, R4007.2, R4011.1
- new net BST_3V3: C4002.1, U4001.6 (BST)
- new net DC_SCM_12V_AUX: C4001.2, R4001.2, R4004.2, U4001.3 (VIN)
- new net DC_SCM_STBY_EN: R4003.1, R4016.1
- new net EN_3V3: R4003.2, R4004.1, R4005.2, U4001.5 (EN)
- new net FB_3V3: R4007.1, R4009.2, U4001.4 (FB)
- new net GND: C4001.1, C4003.1, C4004.1, C4005.1, C4006.1, D4001.1 (C), D4003.1 (C), Q4001.2 (S), R4005.1, R4009.1, R4014.1, R4018.1, U4001.1 (GND), U4002.3 (GND), U4002.5 (GND), U4002.7 (PAD)
- new net SW_3V3: C4002.2, L4001.1, U4001.2 (SW)
Other:
- note added: "+1V8 LDO"
- note added: "+3V3 DC/DC converter"
- note added: "3V3 @ 3A"
- note added: "Note: Vout=0.8V*(1+200k/160k)=1.8V"
- note added: "Status LEDs"

Commit message: chore: set date and project name
Other:
- company: (none) -> Antmicro
- title: (none) -> eSPI Adapter
Changed lines of the file:
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@@
 	(generator_version "10.0")
 	(paper "A4")
+	(title_block
+		(title "eSPI Adapter")
+		(date "2026-08-21")
+		(rev "1.0.0")
+		(company "Antmicro")
+	)
 	(text "Note:\nVout=0.8V*(1+200k/160k)=1.8V"
 		(exclude_from_sim no)
