File: power.kicad_sch (KiCad schematic)
At the start: 31 parts, among them Q4001 DMG1012T-7, U4001 AP62301_TSOT, U4002 TLV76701_WSON

Commit message: [#103753] Fix issues according to the review, add redundant LEDs, delete fp-lib-table
Parts:
- R4002, R4006: now not fitted
Changed lines of the file:
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@@
 		(on_board yes)
 		(in_pos_files yes)
-		(dnp no)
+		(dnp yes)
 		(fields_autoplaced yes)
 		(property "Reference" "R4002"
@@
 		(on_board yes)
 		(in_pos_files yes)
-		(dnp no)
+		(dnp yes)
 		(fields_autoplaced yes)
 		(property "Reference" "R4006"

Commit message: [#103753] Update symbol libraries
Parts:
- R4002, R4006: symbol Antmicro Symbols:R_1k_0402 -> antmicroResistors0402:R_1k_0402

Commit message: [#103697] Reenumerate the entire schematic, rerouting eSPI to maintain bigger gap between traces, rerouting the LDO
Parts:
- renumbered C4005 to C17, C4001 to C18, C4006 to C19, C4002 to C20, C4003 to C21, C4004 to C22, D4001 to D3, D4003 to D4, D4004 to D5, L4001 to L1, Q4001 to Q1, R4016 to R55, R4017 to R56, R4018 to R57, R4012 to R58, R4013 to R59, R4014 to R60, R4015 to R61, R4003 to R62, R4004 to R63, R4005 to R64, R4007 to R65, R4009 to R66, R4001 to R67, R4011 to R68, R4002 to R69, R4006 to R70, TP4002 to TP18, TP4001 to TP19, U4002 to U2, U4001 to U3

Commit message: [#103697] switch dc-dc for TPS566231PRQFR, eSPI length tuning, change zone clearance, fix clearance problems
Parts:
- removed C18: C_10u_16V_0603, antmicro-footprints:C_0603_1608Metric, symbol antmicroCapacitors0603:C_10u_16V_0603
- removed C20: C_100n_50V_X8L_0402, antmicro-footprints:C_0402_1005Metric, symbol antmicroCapacitors0402:C_100n_50V_X8L_0402
- removed C21: C_22u_16V_0603, antmicro-footprints:C_0603_1608Metric_EIA, symbol antmicroCapacitors0603:C_22u_16V_0603
- removed C22: C_22u_0603, antmicro-footprints:C_0603_1608Metric, symbol antmicroCapacitors0603:C_22u_0603
- removed L1: L_3u3_6.6A_XEL4030, antmicro-footprints:L_Coilcraft-XEL4030, symbol antmicroFixedInductors:L_3u3_6.6A_XEL4030
- removed R64, R66: R_10k_0402, antmicro-footprints:R_0402_1005Metric, symbol antmicroResistors0402:R_10k_0402
- removed R65: R_31k6_0402, antmicro-footprints:R_0402_1005Metric, symbol antmicroResistors0402:R_31k6_0402
- removed R68: R_0R_22.4A_0603, antmicro-footprints:R_0603_1608Metric, symbol antmicroResistors0603:R_0R_22.4A_0603
- removed U3: AP62301_TSOT, antmicro-footprints:TSOT23-6, symbol antmicroDCDCConverters:AP62301_TSOT
- added C18, C19, C26, C27, C28: C_22u_16V_0603, antmicro-footprints:C_0603_1608Metric_EIA, symbol antmicroCapacitors0603:C_22u_16V_0603
- added C20, C23, C25: C_100n_0402, antmicro-footprints:C_0402_1005Metric, symbol antmicroCapacitors0402:C_100n_0402
- added C22: C_1u_25V_0402, antmicro-footprints:C_0402_1005Metric, symbol antmicroCapacitors0402:C_1u_25V_0402
- added C24: C_33p_0402, antmicro-footprints:C_0402_1005Metric, symbol antmicroCapacitors0402:C_33p_0402
- added L1: L_2u2_5.8A_WE-PMFI-35329222, antmicro-footprints:L_WE-PMFI-353220, symbol antmicroFixedInductors:L_2u2_5.8A_WE-PMFI-35329222
- added R64: R_100k_0402, antmicro-footprints:R_0402_1005Metric, symbol antmicroResistors0402:R_100k_0402
- added R65: R_10k_0402, antmicro-footprints:R_0402_1005Metric, symbol antmicroResistors0402:R_10k_0402
- added R66: R_135k_0402, antmicro-footprints:R_0402_1005Metric, symbol antmicroResistors0402:R_135k_0402
- added R67: R_30k_0402, antmicro-footprints:R_0402_1005Metric, symbol antmicroResistors0402:R_30k_0402
- added R70: R_0R_22.4A_0603, antmicro-footprints:R_0603_1608Metric, symbol antmicroResistors0603:R_0R_22.4A_0603
- added U3: TPS566231P, antmicro-footprints:VQFN-HR-9_2x1.5mm, symbol antmicroDCDCConverters:TPS566231P
- R62: now not fitted; now in the parts list
- R63: now fitted
- renumbered C19 to C21, R67 to R68, R70 to R71
Connections:
- net +3V3: now also R70.2; no longer TP19.1
- net DC_SCM_12V_AUX: now also C18.2, C19.2, C20.2, U3.5 (V_{IN}), U3.6 (V_{IN})
- net EN_3V3: now also R65.2, U3.3 (EN)
- net GND: now also C18.1, C19.1, C20.1, C22.1, C25.1, C26.1, C27.1, C28.1, R65.1, R67.1, U3.4 (PGND)
- new net +3V3_OUT: C24.2, C25.2, C26.2, C27.2, C28.2, L1.2, R66.2, R70.1, TP19.1
- new net 3V3_BST: C23.1, U3.7 (BST)
- new net 3V3_FB: C24.1, R66.1, R67.2, U3.2 (FB)
- new net 3V3_PG: R64.1, U3.9 (PG)
- new net 3V3_SW: C23.2, L1.1, U3.8 (SW)
- new net 3V3_VCC: C22.2, R64.2, U3.1 (V_{CC})
Other:
- note added: "5V internal LDO"

Commit message: [#103697] Change LDO layout, add power from USB, fix length tuning, change In4.Cu to GND/SIG and In5.Cu to 3V3, cleanup the design
Parts:
- added D16: B340A-13-F, antmicro-footprints:D_SMA, symbol antmicroDiodesRectifiersSingle:B340A-13-F
Connections:
- net DC_SCM_12V_AUX: now also D16.1 (C)
- new net VBUS: D16.2 (A)
Changed lines of the file:
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@@
+	(wire
+		(pts
+			(xy 83.82 38.1) (xy 86.36 38.1)
+		)
+		(stroke
+			(width 0)
+			(type default)
+		)
+	)
 	(wire
 		(pts
@@
 	(wire
 		(pts
+			(xy 86.36 38.1) (xy 86.36 46.99)
+		)
+		(stroke
+			(width 0)
+			(type default)
+		)
+	)
+	(wire
+		(pts
 			(xy 233.68 149.86) (xy 233.68 151.13)
 		)
@@
 		(pts
 			(xy 149.86 62.23) (xy 147.32 62.23)
+		)
+		(stroke
+			(width 0)
+			(type default)
+		)
+	)
+	(wire
+		(pts
+			(xy 72.39 38.1) (xy 78.74 38.1)
 		)
 		(stroke
@@
 		(shape input)
 		(at 195.58 135.89 180)
+		(effects
+			(font
+				(size 1.27 1.27)
+			)
+			(justify right)
+		)
+	)
+	(hierarchical_label "VBUS"
+		(shape input)
+		(at 72.39 38.1 180)
 		(effects
 			(font
@@
 					(unit 1)
 				)
+			)
+		)
+	)
+	(symbol
+		(lib_id "antmicroDiodesRectifiersSingle:B340A-13-F")
+		(at 83.82 38.1 180)
+		(unit 1)
+		(body_style 1)
+		(exclude_from_sim no)
+		(in_bom yes)
+		(on_board yes)
+		(in_pos_files yes)
+		(dnp no)
+		(fields_autoplaced yes)
+		(property "Reference" "D16"
+			(at 81.28 31.75 0)
+			(show_name no)
+			(do_not_autoplace no)
+			(effects
+				(font
+					(size 1.27 1.27)
+					(thickness 0.15)
+				)
+			)
+		)
+		(property "Value" "B340A-13-F"
+			(at 68.58 20.32 0)
+			(hide yes)
+			(show_name no)
+			(do_not_autoplace no)
+			(effects
+				(font
+					(size 1.27 1.27)
+					(thickness 0.15)
+				)
+				(justify left bottom)
+			)
+		)
+		(property "Footprint" "antmicro-footprints:D_SMA"
+			(at 68.58 17.78 0)
+			(hide yes)
+			(show_name no)
+			(do_not_autoplace no)
+			(effects
+				(font
+					(size 1.27 1.27)
+					(thickness 0.15)
+				)
+				(justify left bottom)
+			)
+		)
+		(property "Datasheet" "https://www.diodes.com/assets/Datasheets/ds30891.pdf"
+			(at 68.58 15.24 0)
+			(hide yes)
+			(show_name no)
+			(do_not_autoplace no)
+			(effects
+				(font
+					(size 1.27 1.27)
+					(thickness 0.15)
+				)
+				(justify left bottom)
+			)
+		)
+		(property "Description" "Schottky Diode, 40V, 3A, Single"
+			(at 68.58 12.7 0)
+			(hide yes)
+			(show_name no)
+			(do_not_autoplace no)
+			(effects
+				(font
+					(size 1.27 1.27)
+				)
+				(justify left bottom)
+			)
+		)
+		(property "MPN" "B340A-13-F"
+			(at 81.28 34.29 0)
+			(show_name no)
+			(do_not_autoplace no)
+			(effects
+				(font
+					(size 1.27 1.27)
+					(thickness 0.15)
+				)
+			)
+		)
+		(property "Manufacturer" "Diodes Incorporated"
+			(at 68.58 27.94 0)
+			(hide yes)
+			(show_name no)
+			(do_not_autoplace no)
+			(effects
+				(font
+					(size 1.27 1.27)
+					(thickness 0.15)
+				)
+				(justify left bottom)
+			)
+		)
+		(property "License" "Apache-2.0"
+			(at 68.58 25.4 0)
+			(hide yes)
+			(show_name no)
+			(do_not_autoplace no)
+			(effects
+				(font
+					(size 1.27 1.27)
+					(thickness 0.15)
+				)
+				(justify left bottom)
+			)
+		)
+		(property "Author" "Antmicro"
+			(at 68.58 22.86 0)
+			(hide yes)
+			(show_name no)
+			(do_not_autoplace no)
+			(effects
+				(font
+					(size 1.27 1.27)
+					(thickness 0.15)
+				)
+				(justify left bottom)
+			)
+		)
+		(pin "2"
+		)
+		(pin "1"
+		)
+		(instances
+			(project "dc-scm-server-integration-espi-adapter"
+				(path "/df391740-647e-4ab6-9dcd-d61184d66fe9/1d07191d-71e0-43c8-9a4f-6404f7e36093"
+					(reference "D16")
+					(unit 1)
+				)

Commit message: [#103697] pro: update name
Other:
- title: eSPI Adapter -> MEC1723 eSPI Debugger
