File: dc-scm-server-integration-espi-adapter.kicad_pcb (KiCad board)
At the start: 8 copper layers, 90 x 38 mm, 3 parts, among them J10 PinHeader_2x5_P2.54mm_SMD, J17 PinHeader_2x5_P2.54mm_SMD, J5 PinHeader_2x5_P2.54mm_SMD

Commit message: [#103224] Add notes to schematic, fix typos, fix gpio connections, bump date
Other:
- board text removed: "Board outline from debug interposer"
Changed lines of the file:
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@@
 		(layer "Edge.Cuts")
-	)
-	(gr_text "Board outline from debug interposer"
-		(at 102.99 56.37 0)
-		(layer "Dwgs.User")
-		(effects
-			(font
-				(size 1 1)
-				(thickness 0.15)
-			)
-			(justify left bottom)
-		)
 	)
 	(table

Commit message: [103224] Add USB with FT232RL, transfer elements onto PCB, start positioning elements
Parts:
- removed J10, J17, J5: PinHeader_2x5_P2.54mm_SMD, antmicro-footprints:PinHeader_2x5_P2.54mm_SMD
- added C3001: C_1u_0603, antmicro-footprints:C_0603_1608Metric, F.Cu at (74.6, 145.6)
- added C3002: C_22p_0402, antmicro-footprints:C_0402_1005Metric, F.Cu at (78.7, 134.8)
- added C3003: C_22p_0402, antmicro-footprints:C_0402_1005Metric, F.Cu at (76.7, 134.9)
- added C3004: C_100n_0402, antmicro-footprints:C_0402_1005Metric, F.Cu at (36.5, 178.5)
- added C3005: C_100n_0402, antmicro-footprints:C_0402_1005Metric, F.Cu at (36.5, 180.4)
- added C3006: C_100n_0402, antmicro-footprints:C_0402_1005Metric, F.Cu at (36.5, 182.4)
- added C3007: C_100n_0402, antmicro-footprints:C_0402_1005Metric, F.Cu at (36.5, 184.4)
- added C3008: C_100n_0402, antmicro-footprints:C_0402_1005Metric, F.Cu at (36.5, 186.4)
- added C3009: C_100n_0402, antmicro-footprints:C_0402_1005Metric, F.Cu at (36.5, 188.4)
- added C3010: C_1u_6.3V_X6S_0402, antmicro-footprints:C_0402_1005Metric, F.Cu at (36.5, 190.4)
- added C3011: C_100n_0402, antmicro-footprints:C_0402_1005Metric, F.Cu at (39.4, 174.5)
- added C3012: C_100n_0402, antmicro-footprints:C_0402_1005Metric, F.Cu at (39.4, 176.5)
- added C3013: C_1u_6.3V_X6S_0402, antmicro-footprints:C_0402_1005Metric, F.Cu at (39.4, 178.5)
- added C3014: C_1u_0603, antmicro-footprints:C_0603_1608Metric, F.Cu at (42.4, 194.9)
- added C3015: C_1u_0603, antmicro-footprints:C_0603_1608Metric, F.Cu at (42.4, 197.3)
- added C3016: C_1u_0603, antmicro-footprints:C_0603_1608Metric, F.Cu at (42.4, 199.6)
- added C3017: C_1u_0603, antmicro-footprints:C_0603_1608Metric, F.Cu at (42.4, 202.0)
- added C3018: C_1u_6.3V_X6S_0402, antmicro-footprints:C_0402_1005Metric, F.Cu at (39.4, 180.4)
- added C4001: C_10u_16V_0603, antmicro-footprints:C_0603_1608Metric, F.Cu at (44.9, 117.3)
- added C4002: C_100n_50V_X8L_0402, antmicro-footprints:C_0402_1005Metric, F.Cu at (41.4, 103.6)
- added C4003: C_22u_16V_0603, antmicro-footprints:C_0603_1608Metric_EIA, F.Cu at (40.9, 119.5)
- added C4004: C_22u_0603, antmicro-footprints:C_0603_1608Metric, F.Cu at (40.9, 121.9)
- added C4005: C_10u_10V_0402, antmicro-footprints:C_0402_1005Metric, F.Cu at (125.3, 156.4)
- added C4006: C_10u_10V_0402, antmicro-footprints:C_0402_1005Metric, F.Cu at (123.1, 159.0)
- added C5001: C_100n_0402, antmicro-footprints:C_0402_1005Metric, F.Cu at (72.7, 156.8)
- added C5002: C_100n_0402, antmicro-footprints:C_0402_1005Metric, F.Cu at (88.8, 158.1)
- added C6001: C_100n_0402, antmicro-footprints:C_0402_1005Metric, F.Cu at (91.4, 144.9)
- added C6002: C_100n_0402, antmicro-footprints:C_0402_1005Metric, F.Cu at (91.5, 136.8)
- added C7001: C_10u_10V_X7R_0603, antmicro-footprints:C_0603_1608Metric, F.Cu at (142.9, 186.7)
- added C7002: C_100n_0402, antmicro-footprints:C_0402_1005Metric, F.Cu at (118.0, 222.1)
- added C7003: C_100n_0402, antmicro-footprints:C_0402_1005Metric, F.Cu at (118.0, 224.1)
- added C7004: C_100n_0402, antmicro-footprints:C_0402_1005Metric, F.Cu at (118.0, 226.1)
- added C7005: C_1u_0603, antmicro-footprints:C_0603_1608Metric, F.Cu at (107.9, 234.1)
- added D3001: BAT54-02V-G3-08, antmicro-footprints:SOD-523, F.Cu at (25.2, 208.2)
- added D4001: LED_G_0603_LTST-C190GKT, antmicro-footprints:LED_0603_1608Metric_G, F.Cu at (143.0, 177.8)
- added D4003: LED_G_0603_LTST-C190GKT, antmicro-footprints:LED_0603_1608Metric_G, F.Cu at (134.9, 178.4)
- added D4004: LED_G_0603_LTST-C190GKT, antmicro-footprints:LED_0603_1608Metric_G, F.Cu at (126.1, 178.1)
- added D6001: ACDA02-41SURKWA-F01, antmicro-footprints:ACDA02-41SURKWA-F01, F.Cu at (108.4, 145.0)
- added D7001: TPD2E009_SOT-9X3, antmicro-footprints:SOT-723, F.Cu at (118.7, 213.1)
- added FD1001: Fiducial_1mm_Mask2mm, antmicro-footprints:Fiducial_1mm_Mask2mm, F.Cu at (126.7, 113.1)
- added FD1002: Fiducial_1mm_Mask2mm, antmicro-footprints:Fiducial_1mm_Mask2mm, F.Cu at (126.7, 116.6)
- added FD1003: Fiducial_1mm_Mask2mm, antmicro-footprints:Fiducial_1mm_Mask2mm, F.Cu at (130.2, 113.1)
- added FD1004: Fiducial_1mm_Mask2mm, antmicro-footprints:Fiducial_1mm_Mask2mm, F.Cu at (130.2, 116.6)
- added FD1005: Fiducial_1mm_Mask2mm, antmicro-footprints:Fiducial_1mm_Mask2mm, F.Cu at (133.8, 113.1)
- added FD1006: Fiducial_1mm_Mask2mm, antmicro-footprints:Fiducial_1mm_Mask2mm, F.Cu at (133.8, 116.6)
- added FD1007: Fiducial_1mm_Mask2mm, antmicro-footprints:Fiducial_1mm_Mask2mm, F.Cu at (137.3, 113.1)
- added FD1008: Fiducial_1mm_Mask2mm, antmicro-footprints:Fiducial_1mm_Mask2mm, F.Cu at (137.3, 116.6)
- added J2001: PinSocket_2x10_P2.54mm_SMD, antmicro-footprints:PinSocket_2x10_P2.54mm_SMD, F.Cu at (36.6, 144.3)
- added J2002: PinSocket_2x10_P2.54mm_SMD, antmicro-footprints:PinSocket_2x10_P2.54mm_SMD, F.Cu at (116.5, 105.9)
- added J3001: PinHeader_2x5_P1.27mm_SMD, antmicro-footprints:PinHeader_2x5_P1.27mm_SMD, F.Cu at (15.4, 177.3)
- added J3002: PinHeader_2x5_P1.27mm_SMD, antmicro-footprints:PinHeader_2x5_P1.27mm_SMD, F.Cu at (15.4, 184.8)
- added J3003: PinHeader_2x5_P1.27mm_SMD, antmicro-footprints:PinHeader_2x5_P1.27mm_SMD, F.Cu at (15.4, 192.4)
- added J3004: PinHeader_2x5_P1.27mm_SMD, antmicro-footprints:PinHeader_2x5_P1.27mm_SMD, F.Cu at (15.4, 199.9)
- added J3005: PinHeader_2x5_P1.27mm_SMD, antmicro-footprints:PinHeader_2x5_P1.27mm_SMD, F.Cu at (23.2, 177.3)
- added J3006: PinHeader_2x5_P1.27mm_SMD, antmicro-footprints:PinHeader_2x5_P1.27mm_SMD, F.Cu at (23.2, 184.8)
- added J3007: PinHeader_2x5_P1.27mm_SMD, antmicro-footprints:PinHeader_2x5_P1.27mm_SMD, F.Cu at (23.2, 192.4)
- added J3008: PinHeader_2x5_P1.27mm_SMD, antmicro-footprints:PinHeader_2x5_P1.27mm_SMD, F.Cu at (23.2, 199.9)
- added J3009: PinHeader_2x5_P1.27mm_SMD, antmicro-footprints:PinHeader_2x5_P1.27mm_SMD, F.Cu at (85.6, 123.9)
- added J3010: PinHeader_2x5_P1.27mm_SMD, antmicro-footprints:PinHeader_2x5_P1.27mm_SMD, F.Cu at (31.1, 184.8)
- added J3011: PinHeader_2x5_P1.27mm_SMD, antmicro-footprints:PinHeader_2x5_P1.27mm_SMD, F.Cu at (31.1, 192.4)
- added J5001: Tag-Connect_TC2050-IDC-NL_2x5_P1.27mm, antmicro-footprints:Tag-Connect_TC2050-IDC-NL_2x5_P1.27mm, F.Cu at (80.0, 189.4)
- added J5002: Socket_SOP2-16_ACA-SPI-006-K01_Flash_CUSTOM, antmicro-footprints:Socket_SOP2-16_ACA-SPI-006-K01, F.Cu at (80.7, 159.9)
- added J7001: PinHeader_1x3_P2.54mm_SMD, antmicro-footprints:PinHeader_1x3_P2.54mm_SMD, F.Cu at (112.7, 193.6)
- added J7002: PinHeader_1x3_P2.54mm_SMD, antmicro-footprints:PinHeader_1x3_P2.54mm_SMD, F.Cu at (121.7, 193.6)
- added J7003: Tag-Connect_TC2050-IDC-NL_2x5_P1.27mm, antmicro-footprints:Tag-Connect_TC2050-IDC-NL_2x5_P1.27mm, F.Cu at (135.2, 190.9)
- added J7004: USB-C_GCT_USB4105-GF-A, antmicro-footprints:USB-C_Receptacle_GCT_USB4105-GF-A, F.Cu at (111.7, 216.7)
- added L4001: L_3u3_6.6A_XEL4030, antmicro-footprints:L_Coilcraft-XEL4030, F.Cu at (44.7, 113.0)
- added N1001: antmicro_logo, antmicro-footprints:antmicro-logo, F.Cu at (214.1, 1.66)
- added N1002: oshw_logo, antmicro-footprints:oshw-logo, F.Cu at (136.0, 105.8)
- added Q4001: DMG1012T-7, antmicro-footprints:SOT-523, F.Cu at (124.5, 175.5)
- added R3001: R_10k_0402, antmicro-footprints:R_0402_1005Metric, F.Cu at (39.4, 182.4)
- added R3002: R_100R_0402, antmicro-footprints:R_0402_1005Metric, F.Cu at (39.4, 184.4)
- added R3003: R_1k_0402, antmicro-footprints:R_0402_1005Metric, F.Cu at (39.4, 186.4)
- added R3004: R_0R_0402, antmicro-footprints:R_0402_1005Metric, F.Cu at (39.4, 188.4)
- added R3005: R_10k_0402, antmicro-footprints:R_0402_1005Metric, F.Cu at (39.4, 190.4)
- added R3006: R_100R_0402, antmicro-footprints:R_0402_1005Metric, F.Cu at (42.3, 174.5)
- added R3007: R_4k7_0402, antmicro-footprints:R_0402_1005Metric, F.Cu at (42.3, 176.5)
- added R3008: R_4k7_0402, antmicro-footprints:R_0402_1005Metric, F.Cu at (42.3, 178.5)
- added R3009: R_4k7_0402, antmicro-footprints:R_0402_1005Metric, F.Cu at (42.3, 180.4)
- added R3010: R_4k7_0402, antmicro-footprints:R_0402_1005Metric, F.Cu at (42.3, 182.4)
- added R3011: R_4k7_0402, antmicro-footprints:R_0402_1005Metric, F.Cu at (42.3, 184.4)
- added R3012: R_4k7_0402, antmicro-footprints:R_0402_1005Metric, F.Cu at (42.3, 186.4)
- added R3013: R_4k7_0402, antmicro-footprints:R_0402_1005Metric, F.Cu at (42.3, 188.4)
- added R3014: R_4k7_0402, antmicro-footprints:R_0402_1005Metric, F.Cu at (42.3, 190.4)
- added R3015: R_4k7_0402, antmicro-footprints:R_0402_1005Metric, F.Cu at (45.2, 174.5)
- added R3016: R_4k7_0402, antmicro-footprints:R_0402_1005Metric, F.Cu at (45.2, 176.5)
- added R3017: R_4k7_0402, antmicro-footprints:R_0402_1005Metric, F.Cu at (45.2, 178.5)
- added R3018: R_4k7_0402, antmicro-footprints:R_0402_1005Metric, F.Cu at (45.2, 180.4)
- added R3019: R_4k7_0402, antmicro-footprints:R_0402_1005Metric, F.Cu at (45.2, 182.4)
- added R3020: R_4k7_0402, antmicro-footprints:R_0402_1005Metric, F.Cu at (45.2, 184.4)
- added R3021: R_4k7_0402, antmicro-footprints:R_0402_1005Metric, F.Cu at (45.2, 186.4)
- added R3022: R_4k7_0402, antmicro-footprints:R_0402_1005Metric, F.Cu at (45.2, 188.4)
- added R3023: R_4k7_0402, antmicro-footprints:R_0402_1005Metric, F.Cu at (45.2, 190.4)
- added R3024: R_4k7_0402, antmicro-footprints:R_0402_1005Metric, F.Cu at (48.1, 174.5)
- added R3025: R_10k_0402, antmicro-footprints:R_0402_1005Metric, F.Cu at (48.1, 176.5)
- added R3026: R_10k_0402, antmicro-footprints:R_0402_1005Metric, F.Cu at (48.1, 178.5)
- added R3027: R_100R_0402, antmicro-footprints:R_0402_1005Metric, F.Cu at (48.1, 180.4)
- added R3028: R_0R_0402, antmicro-footprints:R_0402_1005Metric, F.Cu at (48.1, 182.4)
- added R3029: R_10k_0402, antmicro-footprints:R_0402_1005Metric, F.Cu at (48.1, 184.4)
- added R3030: R_10k_0402, antmicro-footprints:R_0402_1005Metric, F.Cu at (48.1, 186.4)
- added R3031: R_10k_0402, antmicro-footprints:R_0402_1005Metric, F.Cu at (48.1, 188.4)
- added R3032: R_10k_0402, antmicro-footprints:R_0402_1005Metric, F.Cu at (48.1, 190.4)
- added R3033: R_10k_0402, antmicro-footprints:R_0402_1005Metric, F.Cu at (51.0, 174.5)
- added R3034: R_10k_0402, antmicro-footprints:R_0402_1005Metric, F.Cu at (51.0, 176.5)
- added R3035: R_10k_0402, antmicro-footprints:R_0402_1005Metric, F.Cu at (51.0, 178.5)
- added R3036: R_10k_0402, antmicro-footprints:R_0402_1005Metric, F.Cu at (51.0, 180.4)
- added R3037: R_1k_0402, antmicro-footprints:R_0402_1005Metric, F.Cu at (51.0, 182.4)
- added R3038: R_100k_0402, antmicro-footprints:R_0402_1005Metric, F.Cu at (51.0, 184.4)
- added R3039: R_100k_0402, antmicro-footprints:R_0402_1005Metric, F.Cu at (51.0, 186.4)
- added R3040: R_100k_0402, antmicro-footprints:R_0402_1005Metric, F.Cu at (51.0, 188.4)
- added R4001: R_10k_0402, antmicro-footprints:R_0402_1005Metric, F.Cu at (146.2, 176.5)
- added R4002: R_1k_0402, antmicro-footprints:R_0402_1005Metric, F.Cu at (134.5, 175.6)
- added R4003: R_0R_0402, antmicro-footprints:R_0402_1005Metric, F.Cu at (45.4, 119.6)
- added R4004: R_10k_0402, antmicro-footprints:R_0402_1005Metric, F.Cu at (50.0, 107.9)
- added R4005: R_10k_0402, antmicro-footprints:R_0402_1005Metric, F.Cu at (46.1, 121.8)
- added R4006: R_1k_0402, antmicro-footprints:R_0402_1005Metric, F.Cu at (127.0, 175.6)
- added R4007: R_31k6_0402, antmicro-footprints:R_0402_1005Metric, F.Cu at (38.6, 113.4)
- added R4009: R_10k_0402, antmicro-footprints:R_0402_1005Metric, F.Cu at (40.4, 115.6)
- added R4011: R_0R_22.4A_0603, antmicro-footprints:R_0603_1608Metric, F.Cu at (45.0, 107.4)
- added R4012: R_100k_0402, antmicro-footprints:R_0402_1005Metric, F.Cu at (134.2, 158.7)
- added R4013: R_100k_0402, antmicro-footprints:R_0402_1005Metric, F.Cu at (134.2, 160.7)
- added R4014: R_160k_0402, antmicro-footprints:R_0402_1005Metric, F.Cu at (134.2, 162.7)
- added R4015: R_0R_0402, antmicro-footprints:R_0402_1005Metric, F.Cu at (37.4, 105.2)
- added R4016: R_0R_0402, antmicro-footprints:R_0402_1005Metric, F.Cu at (123.2, 161.9)
- added R4017: R_10k_0402, antmicro-footprints:R_0402_1005Metric, F.Cu at (123.2, 163.9)
- added R4018: R_10k_0402, antmicro-footprints:R_0402_1005Metric, F.Cu at (123.2, 165.9)
- added R5001: R_10k_0402, antmicro-footprints:R_0402_1005Metric, F.Cu at (88.8, 155.4)
- added R5002: R_10k_0402, antmicro-footprints:R_0402_1005Metric, F.Cu at (72.7, 163.1)
- added R5003: R_10k_0402, antmicro-footprints:R_0402_1005Metric, F.Cu at (78.8, 184.0)
- added R5004: R_10k_0402, antmicro-footprints:R_0402_1005Metric, F.Cu at (78.8, 186.0)
- added R5005: R_10k_0402, antmicro-footprints:R_0402_1005Metric, F.Cu at (88.6, 164.9)
- added R5006: R_10k_0402, antmicro-footprints:R_0402_1005Metric, F.Cu at (72.7, 155.4)
- added R5008: R_10k_0402, antmicro-footprints:R_0402_1005Metric, F.Cu at (81.7, 186.0)
- added R6001: R_200R_0402, antmicro-footprints:R_0402_1005Metric, F.Cu at (95.1, 145.6)
- added R6002: R_200R_0402, antmicro-footprints:R_0402_1005Metric, F.Cu at (95.1, 146.6)
- added R6003: R_200R_0402, antmicro-footprints:R_0402_1005Metric, F.Cu at (95.1, 147.6)
- added R6004: R_200R_0402, antmicro-footprints:R_0402_1005Metric, F.Cu at (95.1, 148.6)
- added R6005: R_200R_0402, antmicro-footprints:R_0402_1005Metric, F.Cu at (95.1, 149.6)
- added R6006: R_200R_0402, antmicro-footprints:R_0402_1005Metric, F.Cu at (95.1, 150.6)
- added R6007: R_200R_0402, antmicro-footprints:R_0402_1005Metric, F.Cu at (95.1, 151.6)
- added R6008: R_200R_0402, antmicro-footprints:R_0402_1005Metric, F.Cu at (95.1, 152.6)
- added R6009: R_200R_0402, antmicro-footprints:R_0402_1005Metric, F.Cu at (95.1, 137.5)
- added R6010: R_200R_0402, antmicro-footprints:R_0402_1005Metric, F.Cu at (95.1, 138.5)
- added R6011: R_200R_0402, antmicro-footprints:R_0402_1005Metric, F.Cu at (95.1, 139.5)
- added R6012: R_200R_0402, antmicro-footprints:R_0402_1005Metric, F.Cu at (95.1, 140.5)
- added R6013: R_200R_0402, antmicro-footprints:R_0402_1005Metric, F.Cu at (95.1, 141.5)
- added R6014: R_200R_0402, antmicro-footprints:R_0402_1005Metric, F.Cu at (95.1, 142.5)
- added R6015: R_200R_0402, antmicro-footprints:R_0402_1005Metric, F.Cu at (95.1, 143.5)
- added R6016: R_200R_0402, antmicro-footprints:R_0402_1005Metric, F.Cu at (95.1, 144.5)
- added R7001: R_10k_0402, antmicro-footprints:R_0402_1005Metric, F.Cu at (142.6, 188.9)
- added R7002: R_10k_0402, antmicro-footprints:R_0402_1005Metric, F.Cu at (142.6, 190.9)
- added R7003: R_10k_0402, antmicro-footprints:R_0402_1005Metric, F.Cu at (142.6, 192.8)
- added R7004: R_10k_0402, antmicro-footprints:R_0402_1005Metric, F.Cu at (142.6, 194.8)
- added R7005: R_100k_0402, antmicro-footprints:R_0402_1005Metric, F.Cu at (142.6, 196.8)
- added R7006: R_5k1_0402, antmicro-footprints:R_0402_1005Metric, F.Cu at (118.0, 228.1)
- added R7007: R_5k1_0402, antmicro-footprints:R_0402_1005Metric, F.Cu at (118.0, 230.1)
- added R7008: R_10k_0402, antmicro-footprints:R_0402_1005Metric, F.Cu at (118.0, 232.1)
- added SW3001: SW_B3U-1000P_SMD, antmicro-footprints:SW_B3U-1000P_SMD, F.Cu at (37.8, 193.5)
- added SW3002: SW_B3U-1000P_SMD, antmicro-footprints:SW_B3U-1000P_SMD, F.Cu at (37.8, 197.6)
- added SW3003: SW_B3U-1000P_SMD, antmicro-footprints:SW_B3U-1000P_SMD, F.Cu at (37.8, 201.8)
- added TP3001: TP_1mm_SMD, antmicro-footprints:TP_SMD_1mm, F.Cu at (12.5, 204.8)
- added TP3002: TP_1mm_SMD, antmicro-footprints:TP_SMD_1mm, F.Cu at (12.5, 207.0)
- added TP3003: TP_1mm_SMD, antmicro-footprints:TP_SMD_1mm, F.Cu at (12.5, 209.3)
- added TP3004: TP_1mm_SMD, antmicro-footprints:TP_SMD_1mm, F.Cu at (14.7, 204.8)
- added TP3005: TP_1mm_SMD, antmicro-footprints:TP_SMD_1mm, F.Cu at (14.7, 207.0)
- added TP3006: TP_1mm_SMD, antmicro-footprints:TP_SMD_1mm, F.Cu at (14.7, 209.3)
- added TP3007: TP_1mm_SMD, antmicro-footprints:TP_SMD_1mm, F.Cu at (17.0, 204.8)
- added TP3008: TP_1mm_SMD, antmicro-footprints:TP_SMD_1mm, F.Cu at (17.0, 207.0)
- added TP3009: TP_1mm_SMD, antmicro-footprints:TP_SMD_1mm, F.Cu at (17.0, 209.3)
- added TP3010: TP_1mm_SMD, antmicro-footprints:TP_SMD_1mm, F.Cu at (19.2, 204.8)
- added TP3011: TP_1mm_SMD, antmicro-footprints:TP_SMD_1mm, F.Cu at (19.2, 207.0)
- added TP3012: TP_1mm_SMD, antmicro-footprints:TP_SMD_1mm, F.Cu at (19.2, 209.3)
- added TP4001: TP_0.75mm_SMD, antmicro-footprints:TP_SMD_0.75mm, F.Cu at (47.6, 104.3)
- added TP4002: TP_0.75mm_SMD, antmicro-footprints:TP_SMD_0.75mm, F.Cu at (127.6, 162.6)
- added U3001: MEC1723N-B0-I/SZ, antmicro-footprints:BGA-169-144_9x9mm_Layout13x13_P0.7mm, F.Cu at (80.8, 144.2)
- added U4001: AP62301_TSOT, antmicro-footprints:TSOT23-6, F.Cu at (38.0, 109.5)
- added U4002: TLV76701_WSON, antmicro-footprints:WSON-6-1EP_2x2mm_P0.65mm, F.Cu at (128.4, 159.3)
- added U5001: MT25QU01GBBB8_SOIC, antmicro-footprints:SOIC-16_W7.5mm, F.Cu at (80.7, 159.9)
- added U6001: SN74AC7541_VQFN, antmicro-footprints:VQFN-20_1EP_4.5x2.5mm_P0.5mm, F.Cu at (90.8, 140.3)
- added U6009: SN74AC7541_VQFN, antmicro-footprints:VQFN-20_1EP_4.5x2.5mm_P0.5mm, F.Cu at (90.7, 148.3)
- added U7001: FT232RL, Package_SO:SSOP-28_5.3x10.2mm_P0.65mm, F.Cu at (111.3, 227.0)
- added Y3001: Resonator_32.768kHz_ECX-31B, antmicro-footprints:Resonator_SMD_ECS_ECX-31B_3.2x1.5x0.9mm, F.Cu at (77.7, 136.8)
Other:
- outline, holes or cut-outs redrawn
- board text added: "Proposed board outline matching with DC-SCM interposer board"

Commit message: [#103224] Initial placement/visualization
Parts:
- removed J2001, J2002: PinSocket_2x10_P2.54mm_SMD, antmicro-footprints:PinSocket_2x10_P2.54mm_SMD
- removed J7001: PinHeader_1x3_P2.54mm_SMD, antmicro-footprints:PinHeader_1x3_P2.54mm_SMD
- added H1001: Spacer_Drill4.4mm_H6mm_9774060360R, antmicro-footprints:Spacer_Drill4.4mm_H6mm_9774060360R, F.Cu at (41.0, 129.0)
- added H1002: Spacer_Drill4.4mm_H6mm_9774060360R, antmicro-footprints:Spacer_Drill4.4mm_H6mm_9774060360R, F.Cu at (41.1, 168.0)
- added H1003: Spacer_Drill4.4mm_H6mm_9774060360R, antmicro-footprints:Spacer_Drill4.4mm_H6mm_9774060360R, F.Cu at (123.0, 168.0)
- added H1004: Spacer_Drill4.4mm_H6mm_9774060360R, antmicro-footprints:Spacer_Drill4.4mm_H6mm_9774060360R, F.Cu at (123.0, 129.0)
- added J2003: PinSocket_2x8_P2.54mm_SMD, antmicro-footprints:PinSocket_2x8_P2.54mm_SMD, F.Cu at (45.3, 144.1)
- moved N1001 312.3 mm to (-70.7, 129.7)
- moved C7005 186.4 mm to (130.4, 49.0)
- moved C7001 170.9 mm to (70.3, 32.0)
- moved R7002 170.9 mm to (70.0, 36.2)
- moved R7005 170.9 mm to (70.0, 42.1)
- moved R7003 170.9 mm to (70.0, 38.1)
- moved R7004 170.9 mm to (70.0, 40.1)
- moved C7002 170.1 mm to (129.8, 52.4)
- moved C7003 170.1 mm to (129.8, 54.4)
- moved R7006 170.1 mm to (129.8, 58.4)
- moved R7007 170.1 mm to (129.8, 60.4)
- moved C7004 170.1 mm to (129.8, 56.4)
- moved D7001 170.1 mm to (130.5, 43.4)
- moved R7008 170.1 mm to (129.8, 62.3)
- moved D4003 167.3 mm to (26.4, 51.1)
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Other:
- board size 90 x 38 mm -> 90 x 47 mm
