File: dc-scm-server-integration-espi-adapter.kicad_pcb (KiCad board)
At the start: 8 copper layers, 62 x 87 mm, 234 parts, among them J2001 PinHeader_2x6_P2.54mm_Drill1.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, J3001 PinHeader_2x5_P1.27mm_SMD, J3002 PinHeader_2x5_P1.27mm_SMD, J3003 PinHeader_2x5_P1.27mm_SMD, J3004 PinHeader_2x5_P1.27mm_SMD, J3005 PinHeader_2x5_P1.27mm_SMD, J3006 PinHeader_2x5_P1.27mm_SMD, J3007 PinHeader_2x5_P1.27mm_SMD, J3008 PinHeader_2x5_P1.27mm_SMD, J3009 PinHeader_2x5_P1.27mm_SMD, J3010 PinHeader_2x5_P1.27mm_SMD, J3011 PinHeader_2x5_P1.27mm_SMD, J5001 Tag-Connect_TC2050-IDC-NL_2x5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, J7003 Tag-Connect_TC2050-IDC-NL_2x5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, J7004 USB-C_GCT_USB4105-GF-A, Q4001 DMG1012T-7, SW3001 SW_KSC441J70SHLFS_SMD, SW3002 SW_KSC441J70SHLFS_SMD, SW3004 SW_KSC441J70SHLFS_SMD, U3001 MEC1723N-B0-I/SZ, U4001 AP62301_TSOT, U4002 TLV76701_WSON, U5001 MT25QU01GBBB8_SOIC, U6001 SN74AC7541_VQFN, U6009 SN74AC7541_VQFN, U7002 FT2232HL-REEL, Y3001 Resonator_32.768kHz_ECX-31B, Y7001 Resonator_12MHz_KX-7

Commit message: [#103753] Fixed issues according to the review
Parts:
- turned D4001 to 0 degrees
Routing:
- net /DC-SCM Interposer connector/DC_SCM_STBY_EN: track 6.22 -> 43.6 mm, vias 0 -> 1
- net /Power/EN_3V3: track 2.51 -> 12.6 mm, vias 0 -> 2
- net /Power/BST_3V3: track 0.00 -> 1.36 mm
- net Net-(D4003-A): track 0.00 -> 1.23 mm
- net Net-(D4004-A): track 0.00 -> 1.18 mm
- net Net-(D4001-A): track 0.00 -> 0.65 mm
- added copper zone on F.Cu, net /Power/SW_3V3
