File: connectors.kicad_sch (KiCad schematic)
At the start: 36 parts, among them J7003 Tag-Connect_TC2050-IDC-NL_2x5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, J7004 USB-C_GCT_USB4105-GF-A, U7002 FT2232HL-REEL, Y7001 Resonator_12MHz_KX-7

Commit message: [#103697] Reenumerate the entire schematic, rerouting eSPI to maintain bigger gap between traces, rerouting the LDO
Parts:
- renumbered C7009 to C27, C7013 to C28, C7008 to C29, C7018 to C30, C7012 to C31, C7007 to C32, C7020 to C33, C7017 to C34, C7010 to C35, C7006 to C36, C7003 to C37, C7019 to C38, C7016 to C39, C7011 to C40, C7001 to C41, C7002 to C42, C7021 to C43, D7001 to D15, J7003 to J14, J7004 to J15, R7006 to R100, R7007 to R101, R7013 to R102, R7012 to R103, R7001 to R104, R7002 to R105, R7003 to R106, R7004 to R107, R7005 to R108, R7009 to R109, R7008 to R110, R7014 to R111, R7015 to R112, R7016 to R113, U7002 to U7, Y7001 to Y2

Commit message: [#103697] switch dc-dc for TPS566231PRQFR, eSPI length tuning, change zone clearance, fix clearance problems
Parts:
- renumbered C27 to C33, C28 to C34, C29 to C35, C30 to C36, C31 to C37, C32 to C38, C33 to C39, C34 to C40, C35 to C41, C36 to C42, C37 to C43, C38 to C44, C39 to C45, C40 to C46, C41 to C47, C42 to C48, C43 to C49, R100 to R101, R101 to R102, R102 to R103, R103 to R104, R104 to R105, R105 to R106, R106 to R107, R107 to R108, R108 to R109, R109 to R110, R110 to R111, R111 to R112, R112 to R113, R113 to R114

Commit message: [#103697] Change LDO layout, add power from USB, fix length tuning, change In4.Cu to GND/SIG and In5.Cu to 3V3, cleanup the design
Connections:
- net VBUS: now reaches J15.A4 (VBUS), J15.A9 (VBUS), J15.B4 (VBUS), J15.B9 (VBUS), R103.2
Changed lines of the file:
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@@
+	)
+	(junction
+		(at 90.17 119.38)
+		(diameter 0)
+		(color 0 0 0 0)
 	)
 	(junction
@@
 	(wire
 		(pts
+			(xy 90.17 119.38) (xy 90.17 123.19)
+		)
+		(stroke
+			(width 0)
+			(type default)
+		)
+	)
+	(wire
+		(pts
 			(xy 171.45 85.09) (xy 171.45 71.12)
 		)
@@
 	(wire
 		(pts
-			(xy 90.17 119.38) (xy 90.17 123.19)
-		)
-		(stroke
-			(width 0)
-			(type default)
-		)
-	)
-	(wire
-		(pts
 			(xy 190.5 168.91) (xy 193.04 168.91)
 		)
@@
 	(wire
 		(pts
-			(xy 64.77 119.38) (xy 90.17 119.38)
-		)
-		(stroke
-			(width 0)
-			(type default)
-		)
-	)
-	(wire
-		(pts
 			(xy 33.02 46.99) (xy 57.15 46.99)
 		)
@@
 	(wire
 		(pts
+			(xy 90.17 119.38) (xy 64.77 119.38)
+		)
+		(stroke
+			(width 0)
+			(type default)
+		)
+	)
+	(wire
+		(pts
 			(xy 162.56 134.62) (xy 162.56 120.65)
 		)
@@
 		(pts
 			(xy 156.21 100.33) (xy 193.04 100.33)
+		)
+		(stroke
+			(width 0)
+			(type default)
+		)
+	)
+	(wire
+		(pts
+			(xy 93.98 119.38) (xy 90.17 119.38)
 		)
 		(stroke
@@
 		)
 	)
+	(hierarchical_label "VBUS"
+		(shape output)
+		(at 93.98 119.38 0)
+		(effects
+			(font
+				(size 1.27 1.27)
+			)
+			(justify left)
+		)
+	)

Commit message: [#103697] pro: update name
Other:
- title: eSPI Adapter -> MEC1723 eSPI Debugger
