File: dc-scm-interposer-connector.kicad_sch (KiCad schematic)
At the start: 19 parts, among them J2001 PinHeader_2x6_P2.54mm_Drill1.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

Commit message: [#103697] Reenumerate the entire schematic, rerouting eSPI to maintain bigger gap between traces, rerouting the LDO
Parts:
- renumbered J2001 to J1, R2005 to R1, R2006 to R2, R2007 to R3, R2008 to R4, R2001 to R5, R2002 to R6, R2003 to R7, R2004 to R8, TP2002 to TP1, TP2011 to TP10, TP2003 to TP2, TP2004 to TP3, TP2005 to TP4, TP2006 to TP5, TP2007 to TP6, TP2008 to TP7, TP2009 to TP8, TP2010 to TP9
Changed lines of the file:
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@@
 		(in_pos_files yes)
 		(dnp no)
-		(property "Reference" "J2001"
+		(property "Reference" "J1"
 			(at 146.558 79.502 0)
 			(show_name no)
@@
 			(project "dc-scm-server-integration-espi-adapter"
 				(path "/df391740-647e-4ab6-9dcd-d61184d66fe9/dad11b40-64da-40df-af81-feff62248020"
-					(reference "J2001")
+					(reference "J1")
 					(unit 1)
 				)
@@
 		(dnp no)
 		(fields_autoplaced yes)
-		(property "Reference" "TP2005"
+		(property "Reference" "TP4"
 			(at 157.48 128.27 0)
 			(show_name no)
@@
 			(project "dc-scm-server-integration-espi-adapter"
 				(path "/df391740-647e-4ab6-9dcd-d61184d66fe9/dad11b40-64da-40df-af81-feff62248020"
-					(reference "TP2005")
+					(reference "TP4")
 					(unit 1)
 				)
@@
 		(in_pos_files yes)
 		(dnp no)
-		(property "Reference" "R2007"
+		(property "Reference" "R3"
 			(at 111.76 96.012 0)
 			(show_name no)
@@
 			(project "dc-scm-server-integration-espi-adapter"
 				(path "/df391740-647e-4ab6-9dcd-d61184d66fe9/dad11b40-64da-40df-af81-feff62248020"
-					(reference "R2007")
+					(reference "R3")
 					(unit 1)
 				)
@@
 		(in_pos_files yes)
 		(dnp no)
-		(property "Reference" "R2003"
+		(property "Reference" "R7"
 			(at 191.516 96.012 0)
 			(show_name no)
@@
 			(project "dc-scm-server-integration-espi-adapter"
 				(path "/df391740-647e-4ab6-9dcd-d61184d66fe9/dad11b40-64da-40df-af81-feff62248020"
-					(reference "R2003")
+					(reference "R7")
 					(unit 1)
 				)
@@
 		(dnp no)
 		(fields_autoplaced yes)
-		(property "Reference" "TP2009"
+		(property "Reference" "TP8"
 			(at 157.48 143.51 0)
 			(show_name no)
@@
 			(project "dc-scm-server-integration-espi-adapter"
 				(path "/df391740-647e-4ab6-9dcd-d61184d66fe9/dad11b40-64da-40df-af81-feff62248020"
-					(reference "TP2009")
+					(reference "TP8")
 					(unit 1)
 				)
@@
 		(in_pos_files yes)
 		(dnp no)
-		(property "Reference" "R2004"
+		(property "Reference" "R8"
 			(at 191.516 98.552 0)
 			(show_name no)
@@
 			(project "dc-scm-server-integration-espi-adapter"
 				(path "/df391740-647e-4ab6-9dcd-d61184d66fe9/dad11b40-64da-40df-af81-feff62248020"
-					(reference "R2004")
+					(reference "R8")
 					(unit 1)
 				)
@@
 		(dnp no)
 		(fields_autoplaced yes)
-		(property "Reference" "TP2008"
+		(property "Reference" "TP7"
 			(at 157.48 139.7 0)
 			(show_name no)
@@
 			(project "dc-scm-server-integration-espi-adapter"
 				(path "/df391740-647e-4ab6-9dcd-d61184d66fe9/dad11b40-64da-40df-af81-feff62248020"
-					(reference "TP2008")
+					(reference "TP7")
 					(unit 1)
 				)
@@
 		(in_pos_files yes)
 		(dnp no)
-		(property "Reference" "#PWR2001"
+		(property "Reference" "#PWR02"
 			(at 191.77 86.36 0)
 			(hide yes)
@@
 			(project "dc-scm-server-integration-espi-adapter"
 				(path "/df391740-647e-4ab6-9dcd-d61184d66fe9/dad11b40-64da-40df-af81-feff62248020"
-					(reference "#PWR2001")
+					(reference "#PWR02")
 					(unit 1)
 				)
@@
 		(in_pos_files yes)
 		(dnp no)
-		(property "Reference" "R2001"
+		(property "Reference" "R5"
 			(at 191.516 90.932 0)
 			(show_name no)
@@
 			(project "dc-scm-server-integration-espi-adapter"
 				(path "/df391740-647e-4ab6-9dcd-d61184d66fe9/dad11b40-64da-40df-af81-feff62248020"
-					(reference "R2001")
+					(reference "R5")
 					(unit 1)
 				)
@@
 		(dnp no)
 		(fields_autoplaced yes)
-		(property "Reference" "TP2011"
+		(property "Reference" "TP10"
 			(at 157.48 151.13 0)
 			(show_name no)
@@
 			(project "dc-scm-server-integration-espi-adapter"
 				(path "/df391740-647e-4ab6-9dcd-d61184d66fe9/dad11b40-64da-40df-af81-feff62248020"
-					(reference "TP2011")
+					(reference "TP10")
 					(unit 1)
 				)
@@
 		(dnp no)
 		(fields_autoplaced yes)
-		(property "Reference" "TP2004"
+		(property "Reference" "TP3"
 			(at 157.48 124.46 0)
 			(show_name no)
@@
 			(project "dc-scm-server-integration-espi-adapter"
 				(path "/df391740-647e-4ab6-9dcd-d61184d66fe9/dad11b40-64da-40df-af81-feff62248020"
-					(reference "TP2004")
+					(reference "TP3")
 					(unit 1)
 				)
@@
 		(dnp no)
 		(fields_autoplaced yes)
-		(property "Reference" "TP2010"
+		(property "Reference" "TP9"
 			(at 157.48 147.32 0)
 			(show_name no)
@@
 			(project "dc-scm-server-integration-espi-adapter"
 				(path "/df391740-647e-4ab6-9dcd-d61184d66fe9/dad11b40-64da-40df-af81-feff62248020"
-					(reference "TP2010")
+					(reference "TP9")
 					(unit 1)
 				)
@@
 		(dnp no)
 		(fields_autoplaced yes)
-		(property "Reference" "TP2007"
+		(property "Reference" "TP6"
 			(at 157.48 135.89 0)
 			(show_name no)
@@
 			(project "dc-scm-server-integration-espi-adapter"
 				(path "/df391740-647e-4ab6-9dcd-d61184d66fe9/dad11b40-64da-40df-af81-feff62248020"
-					(reference "TP2007")
+					(reference "TP6")
 					(unit 1)
 				)
@@
 		(dnp no)
 		(fields_autoplaced yes)
-		(property "Reference" "TP2006"
+		(property "Reference" "TP5"
 			(at 157.48 132.08 0)
 			(show_name no)
@@
 			(project "dc-scm-server-integration-espi-adapter"
 				(path "/df391740-647e-4ab6-9dcd-d61184d66fe9/dad11b40-64da-40df-af81-feff62248020"
-					(reference "TP2006")
+					(reference "TP5")
 					(unit 1)
 				)
@@
 		(dnp no)
 		(fields_autoplaced yes)
-		(property "Reference" "TP2002"
+		(property "Reference" "TP1"
 			(at 157.48 115.57 0)
 			(show_name no)
@@
 			(project "dc-scm-server-integration-espi-adapter"
 				(path "/df391740-647e-4ab6-9dcd-d61184d66fe9/dad11b40-64da-40df-af81-feff62248020"
-					(reference "TP2002")
+					(reference "TP1")
 					(unit 1)
 				)
@@
 		(in_pos_files yes)
 		(dnp no)
-		(property "Reference" "R2006"
+		(property "Reference" "R2"
 			(at 111.506 93.472 0)
 			(show_name no)
@@
 			(project "dc-scm-server-integration-espi-adapter"
 				(path "/df391740-647e-4ab6-9dcd-d61184d66fe9/dad11b40-64da-40df-af81-feff62248020"
-					(reference "R2006")
+					(reference "R2")
 					(unit 1)
 				)
@@
 		(dnp no)
 		(fields_autoplaced yes)
-		(property "Reference" "TP2003"
+		(property "Reference" "TP2"
 			(at 157.48 119.38 0)
 			(show_name no)
@@
 			(project "dc-scm-server-integration-espi-adapter"
 				(path "/df391740-647e-4ab6-9dcd-d61184d66fe9/dad11b40-64da-40df-af81-feff62248020"
-					(reference "TP2003")
+					(reference "TP2")
 					(unit 1)
 				)
@@
 		(in_pos_files yes)
 		(dnp no)
-		(property "Reference" "R2005"
+		(property "Reference" "R1"
 			(at 111.506 90.678 0)
 			(show_name no)
@@
 			(project "dc-scm-server-integration-espi-adapter"
 				(path "/df391740-647e-4ab6-9dcd-d61184d66fe9/dad11b40-64da-40df-af81-feff62248020"
-					(reference "R2005")
+					(reference "R1")
 					(unit 1)
 				)
@@
 		(in_pos_files yes)
 		(dnp no)
-		(property "Reference" "R2008"
+		(property "Reference" "R4"
 			(at 111.76 98.806 0)
 			(show_name no)
@@
 			(project "dc-scm-server-integration-espi-adapter"
 				(path "/df391740-647e-4ab6-9dcd-d61184d66fe9/dad11b40-64da-40df-af81-feff62248020"
-					(reference "R2008")
+					(reference "R4")
 					(unit 1)
 				)
@@
 		(in_pos_files yes)
 		(dnp no)
-		(property "Reference" "R2002"
+		(property "Reference" "R6"
 			(at 191.516 93.472 0)
 			(show_name no)
@@
 			(project "dc-scm-server-integration-espi-adapter"
 				(path "/df391740-647e-4ab6-9dcd-d61184d66fe9/dad11b40-64da-40df-af81-feff62248020"
-					(reference "R2002")
+					(reference "R6")
 					(unit 1)
 				)

Commit message: [#103697] Change LDO layout, add power from USB, fix length tuning, change In4.Cu to GND/SIG and In5.Cu to 3V3, cleanup the design
Parts:
- removed TP10, TP3, TP4, TP5, TP6, TP7, TP8, TP9: TP_1mm_SMD, antmicro-footprints:TP_SMD_1mm, symbol antmicroTestPoints:TP_1mm_SMD
- added TP10, TP3, TP4, TP5, TP6, TP7, TP8, TP9: TP_0.75mm_SMD, antmicro-footprints:TP_SMD_0.75mm, symbol antmicroTestPoints:TP_0.75mm_SMD
Connections:
- net EC_ESPI.IO0: now also TP6.1
- net EC_ESPI.IO1: now also TP7.1
- net EC_ESPI.IO2: now also TP8.1
- net EC_ESPI.IO3: now also TP9.1
- net EC_ESPI.SCK: now also TP3.1
- net EC_ESPI.~{ALERT0}: now also TP10.1
- net EC_ESPI.~{CS0}: now also TP4.1
- net EC_ESPI.~{RESET}: now also TP5.1

Commit message: [#103697] pro: update name
Other:
- title: eSPI Adapter -> MEC1723 eSPI Debugger
Changed lines of the file:
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@@
 	(paper "A4")
 	(title_block
-		(title "eSPI Adapter")
-		(date "2026-08-21")
+		(title "MEC1723 eSPI Debugger")
+		(date "2026-09-02")
 		(rev "1.0.0")
 		(company "Antmicro")
@@
 		)
 		(instances
-			(project "dc-scm-server-integration-espi-adapter"
+			(project "mec1723-espi-debugger"
 				(path "/df391740-647e-4ab6-9dcd-d61184d66fe9/dad11b40-64da-40df-af81-feff62248020"
 					(reference "TP8")
@@
 		)
 		(instances
-			(project "dc-scm-server-integration-espi-adapter"
+			(project "mec1723-espi-debugger"
 				(path "/df391740-647e-4ab6-9dcd-d61184d66fe9/dad11b40-64da-40df-af81-feff62248020"
 					(reference "J1")
@@
 		)
 		(instances
-			(project "dc-scm-server-integration-espi-adapter"
+			(project "mec1723-espi-debugger"
 				(path "/df391740-647e-4ab6-9dcd-d61184d66fe9/dad11b40-64da-40df-af81-feff62248020"
 					(reference "TP6")
@@
 		)
 		(instances
-			(project "dc-scm-server-integration-espi-adapter"
+			(project "mec1723-espi-debugger"
 				(path "/df391740-647e-4ab6-9dcd-d61184d66fe9/dad11b40-64da-40df-af81-feff62248020"
 					(reference "R3")
@@
 		)
 		(instances
-			(project "dc-scm-server-integration-espi-adapter"
+			(project "mec1723-espi-debugger"
 				(path "/df391740-647e-4ab6-9dcd-d61184d66fe9/dad11b40-64da-40df-af81-feff62248020"
 					(reference "TP5")
@@
 		)
 		(instances
-			(project "dc-scm-server-integration-espi-adapter"
+			(project "mec1723-espi-debugger"
 				(path "/df391740-647e-4ab6-9dcd-d61184d66fe9/dad11b40-64da-40df-af81-feff62248020"
 					(reference "R7")
@@
 		)
 		(instances
-			(project "dc-scm-server-integration-espi-adapter"
+			(project "mec1723-espi-debugger"
 				(path "/df391740-647e-4ab6-9dcd-d61184d66fe9/dad11b40-64da-40df-af81-feff62248020"
 					(reference "R8")
@@
 		)
 		(instances
-			(project "dc-scm-server-integration-espi-adapter"
+			(project "mec1723-espi-debugger"
 				(path "/df391740-647e-4ab6-9dcd-d61184d66fe9/dad11b40-64da-40df-af81-feff62248020"
 					(reference "TP3")
@@
 		)
 		(instances
-			(project "dc-scm-server-integration-espi-adapter"
+			(project "mec1723-espi-debugger"
 				(path "/df391740-647e-4ab6-9dcd-d61184d66fe9/dad11b40-64da-40df-af81-feff62248020"
 					(reference "#PWR02")
@@
 		)
 		(instances
-			(project "dc-scm-server-integration-espi-adapter"
+			(project "mec1723-espi-debugger"
 				(path "/df391740-647e-4ab6-9dcd-d61184d66fe9/dad11b40-64da-40df-af81-feff62248020"
 					(reference "R5")
@@
 		)
 		(instances
-			(project "dc-scm-server-integration-espi-adapter"
+			(project "mec1723-espi-debugger"
 				(path "/df391740-647e-4ab6-9dcd-d61184d66fe9/dad11b40-64da-40df-af81-feff62248020"
 					(reference "TP10")
@@
 		)
 		(instances
-			(project "dc-scm-server-integration-espi-adapter"
+			(project "mec1723-espi-debugger"
 				(path "/df391740-647e-4ab6-9dcd-d61184d66fe9/dad11b40-64da-40df-af81-feff62248020"
 					(reference "TP1")
@@
 		)
 		(instances
-			(project "dc-scm-server-integration-espi-adapter"
+			(project "mec1723-espi-debugger"
 				(path "/df391740-647e-4ab6-9dcd-d61184d66fe9/dad11b40-64da-40df-af81-feff62248020"
 					(reference "R2")
@@
 		)
 		(instances
-			(project "dc-scm-server-integration-espi-adapter"
+			(project "mec1723-espi-debugger"
 				(path "/df391740-647e-4ab6-9dcd-d61184d66fe9/dad11b40-64da-40df-af81-feff62248020"
 					(reference "TP2")
@@
 		)
 		(instances
-			(project "dc-scm-server-integration-espi-adapter"
+			(project "mec1723-espi-debugger"
 				(path "/df391740-647e-4ab6-9dcd-d61184d66fe9/dad11b40-64da-40df-af81-feff62248020"
 					(reference "R1")
@@
 		)
 		(instances
-			(project "dc-scm-server-integration-espi-adapter"
+			(project "mec1723-espi-debugger"
 				(path "/df391740-647e-4ab6-9dcd-d61184d66fe9/dad11b40-64da-40df-af81-feff62248020"
 					(reference "TP9")
@@
 		)
 		(instances
-			(project "dc-scm-server-integration-espi-adapter"
+			(project "mec1723-espi-debugger"
 				(path "/df391740-647e-4ab6-9dcd-d61184d66fe9/dad11b40-64da-40df-af81-feff62248020"
 					(reference "R4")
@@
 		)
 		(instances
-			(project "dc-scm-server-integration-espi-adapter"
+			(project "mec1723-espi-debugger"
 				(path "/df391740-647e-4ab6-9dcd-d61184d66fe9/dad11b40-64da-40df-af81-feff62248020"
 					(reference "TP4")
@@
 		)
 		(instances
-			(project "dc-scm-server-integration-espi-adapter"
+			(project "mec1723-espi-debugger"
 				(path "/df391740-647e-4ab6-9dcd-d61184d66fe9/dad11b40-64da-40df-af81-feff62248020"
 					(reference "R6")
@@
 		)
 		(instances
-			(project "dc-scm-server-integration-espi-adapter"
+			(project "mec1723-espi-debugger"
 				(path "/df391740-647e-4ab6-9dcd-d61184d66fe9/dad11b40-64da-40df-af81-feff62248020"
 					(reference "TP7")
