File: flash.kicad_sch (KiCad schematic)
At the start: 17 parts, among them J5001 Tag-Connect_TC2050-IDC-NL_2x5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, U5001 MT25QU01GBBB8_SOIC

Commit message: [#103697] Reenumerate the entire schematic, rerouting eSPI to maintain bigger gap between traces, rerouting the LDO
Parts:
- renumbered C5001 to C23, C5002 to C24, J5001 to J13, R5001 to R71, R5002 to R72, R5003 to R73, R5004 to R74, R5005 to R75, R5006 to R76, R5007 to R77, R5009 to R78, R5010 to R79, R5011 to R80, R5012 to R81, R5013 to R82, R5008 to R83, U5001 to U4
Changed lines of the file:
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@@
 		(dnp no)
 		(fields_autoplaced yes)
-		(property "Reference" "#PWR5005"
+		(property "Reference" "#PWR096"
 			(at 228.6 88.9 0)
 			(hide yes)
@@
 			(project "dc-scm-server-integration-espi-adapter"
 				(path "/df391740-647e-4ab6-9dcd-d61184d66fe9/870b0b62-f962-4a87-8d30-5a8522c5db60"
-					(reference "#PWR5005")
+					(reference "#PWR096")
 					(unit 1)
 				)
@@
 		(in_pos_files yes)
 		(dnp no)
-		(property "Reference" "#PWR5006"
+		(property "Reference" "#PWR097"
 			(at 238.76 55.88 0)
 			(hide yes)
@@
 			(project "dc-scm-server-integration-espi-adapter"
 				(path "/df391740-647e-4ab6-9dcd-d61184d66fe9/870b0b62-f962-4a87-8d30-5a8522c5db60"
-					(reference "#PWR5006")
+					(reference "#PWR097")
 					(unit 1)
 				)
@@
 		(in_pos_files yes)
 		(dnp no)
-		(property "Reference" "#PWR5004"
+		(property "Reference" "#PWR095"
 			(at 163.83 66.04 0)
 			(hide yes)
@@
 			(project "dc-scm-server-integration-espi-adapter"
 				(path "/df391740-647e-4ab6-9dcd-d61184d66fe9/870b0b62-f962-4a87-8d30-5a8522c5db60"
-					(reference "#PWR5004")
+					(reference "#PWR095")
 					(unit 1)
 				)
@@
 		(in_pos_files yes)
 		(dnp no)
-		(property "Reference" "R5005"
+		(property "Reference" "R75"
 			(at 125.73 58.42 90)
 			(show_name no)
@@
 			(project "dc-scm-server-integration-espi-adapter"
 				(path "/df391740-647e-4ab6-9dcd-d61184d66fe9/870b0b62-f962-4a87-8d30-5a8522c5db60"
-					(reference "R5005")
+					(reference "R75")
 					(unit 1)
 				)
@@
 		(in_pos_files yes)
 		(dnp no)
-		(property "Reference" "#PWR5003"
+		(property "Reference" "#PWR094"
 			(at 187.96 55.88 0)
 			(hide yes)
@@
 			(project "dc-scm-server-integration-espi-adapter"
 				(path "/df391740-647e-4ab6-9dcd-d61184d66fe9/870b0b62-f962-4a87-8d30-5a8522c5db60"
-					(reference "#PWR5003")
+					(reference "#PWR094")
 					(unit 1)
 				)
@@
 		(in_pos_files yes)
 		(dnp no)
-		(property "Reference" "R5007"
+		(property "Reference" "R77"
 			(at 144.526 70.866 0)
 			(show_name no)
@@
 			(project "dc-scm-server-integration-espi-adapter"
 				(path "/df391740-647e-4ab6-9dcd-d61184d66fe9/870b0b62-f962-4a87-8d30-5a8522c5db60"
-					(reference "R5007")
+					(reference "R77")
 					(unit 1)
 				)
@@
 		(dnp no)
 		(fields_autoplaced yes)
-		(property "Reference" "U5001"
+		(property "Reference" "U4"
 			(at 206.375 57.15 0)
 			(show_name no)
@@
 			(project "dc-scm-server-integration-espi-adapter"
 				(path "/df391740-647e-4ab6-9dcd-d61184d66fe9/870b0b62-f962-4a87-8d30-5a8522c5db60"
-					(reference "U5001")
+					(reference "U4")
 					(unit 1)
 				)
@@
 		(in_pos_files yes)
 		(dnp no)
-		(property "Reference" "#PWR5009"
+		(property "Reference" "#PWR093"
 			(at 172.72 127 0)
 			(hide yes)
@@
 			(project "dc-scm-server-integration-espi-adapter"
 				(path "/df391740-647e-4ab6-9dcd-d61184d66fe9/870b0b62-f962-4a87-8d30-5a8522c5db60"
-					(reference "#PWR5009")
+					(reference "#PWR093")
 					(unit 1)
 				)
@@
 		(in_pos_files yes)
 		(dnp no)
-		(property "Reference" "C5001"
+		(property "Reference" "C23"
 			(at 163.576 56.896 90)
 			(show_name no)
@@
 			(project "dc-scm-server-integration-espi-adapter"
 				(path "/df391740-647e-4ab6-9dcd-d61184d66fe9/870b0b62-f962-4a87-8d30-5a8522c5db60"
-					(reference "C5001")
+					(reference "C23")
 					(unit 1)
 				)
@@
 		(in_pos_files yes)
 		(dnp no)
-		(property "Reference" "R5012"
+		(property "Reference" "R81"
 			(at 144.526 81.026 0)
 			(show_name no)
@@
 			(project "dc-scm-server-integration-espi-adapter"
 				(path "/df391740-647e-4ab6-9dcd-d61184d66fe9/870b0b62-f962-4a87-8d30-5a8522c5db60"
-					(reference "R5012")
+					(reference "R81")
 					(unit 1)
 				)
@@
 		(in_pos_files yes)
 		(dnp no)
-		(property "Reference" "R5011"
+		(property "Reference" "R80"
 			(at 144.526 78.486 0)
 			(show_name no)
@@
 			(project "dc-scm-server-integration-espi-adapter"
 				(path "/df391740-647e-4ab6-9dcd-d61184d66fe9/870b0b62-f962-4a87-8d30-5a8522c5db60"
-					(reference "R5011")
+					(reference "R80")
 					(unit 1)
 				)
@@
 		(dnp no)
 		(fields_autoplaced yes)
-		(property "Reference" "C5002"
+		(property "Reference" "C24"
 			(at 226.06 67.3036 90)
 			(show_name no)
@@
 			(project "dc-scm-server-integration-espi-adapter"
 				(path "/df391740-647e-4ab6-9dcd-d61184d66fe9/870b0b62-f962-4a87-8d30-5a8522c5db60"
-					(reference "C5002")
+					(reference "C24")
 					(unit 1)
 				)
@@
 		(in_pos_files yes)
 		(dnp no)
-		(property "Reference" "R5004"
+		(property "Reference" "R74"
 			(at 116.84 58.42 90)
 			(show_name no)
@@
 			(project "dc-scm-server-integration-espi-adapter"
 				(path "/df391740-647e-4ab6-9dcd-d61184d66fe9/870b0b62-f962-4a87-8d30-5a8522c5db60"
-					(reference "R5004")
+					(reference "R74")
 					(unit 1)
 				)
@@
 		(dnp no)
 		(fields_autoplaced yes)
-		(property "Reference" "J5001"
+		(property "Reference" "J13"
 			(at 146.685 104.14 0)
 			(show_name no)
@@
 			(project "dc-scm-server-integration-espi-adapter"
 				(path "/df391740-647e-4ab6-9dcd-d61184d66fe9/870b0b62-f962-4a87-8d30-5a8522c5db60"
-					(reference "J5001")
+					(reference "J13")
 					(unit 1)
 				)
@@
 		(in_pos_files yes)
 		(dnp no)
-		(property "Reference" "R5013"
+		(property "Reference" "R82"
 			(at 144.526 83.566 0)
 			(show_name no)
@@
 			(project "dc-scm-server-integration-espi-adapter"
 				(path "/df391740-647e-4ab6-9dcd-d61184d66fe9/870b0b62-f962-4a87-8d30-5a8522c5db60"
-					(reference "R5013")
+					(reference "R82")
 					(unit 1)
 				)
@@
 		(in_pos_files yes)
 		(dnp no)
-		(property "Reference" "R5009"
+		(property "Reference" "R78"
 			(at 144.526 73.406 0)
 			(show_name no)
@@
 			(project "dc-scm-server-integration-espi-adapter"
 				(path "/df391740-647e-4ab6-9dcd-d61184d66fe9/870b0b62-f962-4a87-8d30-5a8522c5db60"
-					(reference "R5009")
+					(reference "R78")
 					(unit 1)
 				)
@@
 		(in_pos_files yes)
 		(dnp no)
-		(property "Reference" "#PWR5002"
+		(property "Reference" "#PWR091"
 			(at 143.51 111.76 0)
 			(hide yes)
@@
 			(project "dc-scm-server-integration-espi-adapter"
 				(path "/df391740-647e-4ab6-9dcd-d61184d66fe9/870b0b62-f962-4a87-8d30-5a8522c5db60"
-					(reference "#PWR5002")
+					(reference "#PWR091")
 					(unit 1)
 				)
@@
 		(dnp no)
 		(fields_autoplaced yes)
-		(property "Reference" "#PWR5007"
+		(property "Reference" "#PWR098"
 			(at 232.41 74.93 0)
 			(hide yes)
@@
 			(project "dc-scm-server-integration-espi-adapter"
 				(path "/df391740-647e-4ab6-9dcd-d61184d66fe9/870b0b62-f962-4a87-8d30-5a8522c5db60"
-					(reference "#PWR5007")
+					(reference "#PWR098")
 					(unit 1)
 				)
@@
 		(in_pos_files yes)
 		(dnp no)
-		(property "Reference" "#PWR5008"
+		(property "Reference" "#PWR092"
 			(at 138.43 127 0)
 			(hide yes)
@@
 			(project "dc-scm-server-integration-espi-adapter"
 				(path "/df391740-647e-4ab6-9dcd-d61184d66fe9/870b0b62-f962-4a87-8d30-5a8522c5db60"
-					(reference "#PWR5008")
+					(reference "#PWR092")
 					(unit 1)
 				)
@@
 		(in_pos_files yes)
 		(dnp no)
-		(property "Reference" "#PWR5001"
+		(property "Reference" "#PWR090"
 			(at 104.14 55.88 0)
 			(hide yes)
@@
 			(project "dc-scm-server-integration-espi-adapter"
 				(path "/df391740-647e-4ab6-9dcd-d61184d66fe9/870b0b62-f962-4a87-8d30-5a8522c5db60"
-					(reference "#PWR5001")
+					(reference "#PWR090")
 					(unit 1)
 				)
@@
 		(in_pos_files yes)
 		(dnp no)
-		(property "Reference" "R5003"
+		(property "Reference" "R73"
 			(at 107.95 58.42 90)
 			(show_name no)
@@
 			(project "dc-scm-server-integration-espi-adapter"
 				(path "/df391740-647e-4ab6-9dcd-d61184d66fe9/870b0b62-f962-4a87-8d30-5a8522c5db60"
-					(reference "R5003")
+					(reference "R73")
 					(unit 1)
 				)
@@
 		(in_pos_files yes)
 		(dnp no)
-		(property "Reference" "R5010"
+		(property "Reference" "R79"
 			(at 144.526 75.946 0)
 			(show_name no)
@@
 			(project "dc-scm-server-integration-espi-adapter"
 				(path "/df391740-647e-4ab6-9dcd-d61184d66fe9/870b0b62-f962-4a87-8d30-5a8522c5db60"
-					(reference "R5010")
+					(reference "R79")
 					(unit 1)
 				)
@@
 		(in_pos_files yes)
 		(dnp no)
-		(property "Reference" "R5002"
+		(property "Reference" "R72"
 			(at 99.06 58.42 90)
 			(show_name no)
@@
 			(project "dc-scm-server-integration-espi-adapter"
 				(path "/df391740-647e-4ab6-9dcd-d61184d66fe9/870b0b62-f962-4a87-8d30-5a8522c5db60"
-					(reference "R5002")
+					(reference "R72")
 					(unit 1)
 				)
@@
 		(in_pos_files yes)
 		(dnp no)
-		(property "Reference" "R5001"
+		(property "Reference" "R71"
 			(at 90.17 58.42 90)
 			(show_name no)
@@
 			(project "dc-scm-server-integration-espi-adapter"
 				(path "/df391740-647e-4ab6-9dcd-d61184d66fe9/870b0b62-f962-4a87-8d30-5a8522c5db60"
-					(reference "R5001")
+					(reference "R71")
 					(unit 1)
 				)
@@
 		(in_pos_files yes)
 		(dnp no)
-		(property "Reference" "R5008"
+		(property "Reference" "R83"
 			(at 182.88 58.42 90)
 			(show_name no)
@@
 			(project "dc-scm-server-integration-espi-adapter"
 				(path "/df391740-647e-4ab6-9dcd-d61184d66fe9/870b0b62-f962-4a87-8d30-5a8522c5db60"
-					(reference "R5008")
+					(reference "R83")
 					(unit 1)
 				)
@@
 		(in_pos_files yes)
 		(dnp no)
-		(property "Reference" "R5006"
+		(property "Reference" "R76"
 			(at 134.62 58.42 90)
 			(show_name no)
@@
 			(project "dc-scm-server-integration-espi-adapter"
 				(path "/df391740-647e-4ab6-9dcd-d61184d66fe9/870b0b62-f962-4a87-8d30-5a8522c5db60"
-					(reference "R5006")
+					(reference "R76")
 					(unit 1)
 				)

Commit message: [#103697] switch dc-dc for TPS566231PRQFR, eSPI length tuning, change zone clearance, fix clearance problems
Parts:
- renumbered C23 to C29, C24 to C30, R71 to R72, R72 to R73, R73 to R74, R74 to R75, R75 to R76, R76 to R77, R77 to R78, R78 to R79, R79 to R80, R80 to R81, R81 to R82, R82 to R83, R83 to R84
Changed lines of the file:
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@@
 		(dnp no)
 		(fields_autoplaced yes)
-		(property "Reference" "#PWR096"
+		(property "Reference" "#PWR0102"
 			(at 228.6 88.9 0)
 			(hide yes)
@@
 			(project "dc-scm-server-integration-espi-adapter"
 				(path "/df391740-647e-4ab6-9dcd-d61184d66fe9/870b0b62-f962-4a87-8d30-5a8522c5db60"
-					(reference "#PWR096")
+					(reference "#PWR0102")
 					(unit 1)
 				)
@@
 		(in_pos_files yes)
 		(dnp no)
-		(property "Reference" "#PWR097"
+		(property "Reference" "#PWR0103"
 			(at 238.76 55.88 0)
 			(hide yes)
@@
 			(project "dc-scm-server-integration-espi-adapter"
 				(path "/df391740-647e-4ab6-9dcd-d61184d66fe9/870b0b62-f962-4a87-8d30-5a8522c5db60"
-					(reference "#PWR097")
+					(reference "#PWR0103")
 					(unit 1)
 				)
@@
 		(in_pos_files yes)
 		(dnp no)
-		(property "Reference" "#PWR095"
+		(property "Reference" "#PWR0101"
 			(at 163.83 66.04 0)
 			(hide yes)
@@
 			(project "dc-scm-server-integration-espi-adapter"
 				(path "/df391740-647e-4ab6-9dcd-d61184d66fe9/870b0b62-f962-4a87-8d30-5a8522c5db60"
-					(reference "#PWR095")
+					(reference "#PWR0101")
 					(unit 1)
 				)
@@
 		(in_pos_files yes)
 		(dnp no)
-		(property "Reference" "R75"
+		(property "Reference" "R76"
 			(at 125.73 58.42 90)
 			(show_name no)
@@
 			(project "dc-scm-server-integration-espi-adapter"
 				(path "/df391740-647e-4ab6-9dcd-d61184d66fe9/870b0b62-f962-4a87-8d30-5a8522c5db60"
-					(reference "R75")
+					(reference "R76")
 					(unit 1)
 				)
@@
 		(in_pos_files yes)
 		(dnp no)
-		(property "Reference" "#PWR094"
+		(property "Reference" "#PWR0100"
 			(at 187.96 55.88 0)
 			(hide yes)
@@
 			(project "dc-scm-server-integration-espi-adapter"
 				(path "/df391740-647e-4ab6-9dcd-d61184d66fe9/870b0b62-f962-4a87-8d30-5a8522c5db60"
-					(reference "#PWR094")
+					(reference "#PWR0100")
 					(unit 1)
 				)
@@
 		(in_pos_files yes)
 		(dnp no)
-		(property "Reference" "R77"
+		(property "Reference" "R78"
 			(at 144.526 70.866 0)
 			(show_name no)
@@
 			(project "dc-scm-server-integration-espi-adapter"
 				(path "/df391740-647e-4ab6-9dcd-d61184d66fe9/870b0b62-f962-4a87-8d30-5a8522c5db60"
-					(reference "R77")
+					(reference "R78")
 					(unit 1)
 				)
@@
 		(in_pos_files yes)
 		(dnp no)
-		(property "Reference" "#PWR093"
+		(property "Reference" "#PWR099"
 			(at 172.72 127 0)
 			(hide yes)
@@
 			(project "dc-scm-server-integration-espi-adapter"
 				(path "/df391740-647e-4ab6-9dcd-d61184d66fe9/870b0b62-f962-4a87-8d30-5a8522c5db60"
-					(reference "#PWR093")
+					(reference "#PWR099")
 					(unit 1)
 				)
@@
 		(in_pos_files yes)
 		(dnp no)
-		(property "Reference" "C23"
+		(property "Reference" "C29"
 			(at 163.576 56.896 90)
 			(show_name no)
@@
 			(project "dc-scm-server-integration-espi-adapter"
 				(path "/df391740-647e-4ab6-9dcd-d61184d66fe9/870b0b62-f962-4a87-8d30-5a8522c5db60"
-					(reference "C23")
+					(reference "C29")
 					(unit 1)
 				)
@@
 		(in_pos_files yes)
 		(dnp no)
-		(property "Reference" "R81"
+		(property "Reference" "R82"
 			(at 144.526 81.026 0)
 			(show_name no)
@@
 			(project "dc-scm-server-integration-espi-adapter"
 				(path "/df391740-647e-4ab6-9dcd-d61184d66fe9/870b0b62-f962-4a87-8d30-5a8522c5db60"
-					(reference "R81")
+					(reference "R82")
 					(unit 1)
 				)
@@
 		(in_pos_files yes)
 		(dnp no)
-		(property "Reference" "R80"
+		(property "Reference" "R81"
 			(at 144.526 78.486 0)
 			(show_name no)
@@
 			(project "dc-scm-server-integration-espi-adapter"
 				(path "/df391740-647e-4ab6-9dcd-d61184d66fe9/870b0b62-f962-4a87-8d30-5a8522c5db60"
-					(reference "R80")
+					(reference "R81")
 					(unit 1)
 				)
@@
 		(dnp no)
 		(fields_autoplaced yes)
-		(property "Reference" "C24"
+		(property "Reference" "C30"
 			(at 226.06 67.3036 90)
 			(show_name no)
@@
 			(project "dc-scm-server-integration-espi-adapter"
 				(path "/df391740-647e-4ab6-9dcd-d61184d66fe9/870b0b62-f962-4a87-8d30-5a8522c5db60"
-					(reference "C24")
+					(reference "C30")
 					(unit 1)
 				)
@@
 		(in_pos_files yes)
 		(dnp no)
-		(property "Reference" "R74"
+		(property "Reference" "R75"
 			(at 116.84 58.42 90)
 			(show_name no)
@@
 			(project "dc-scm-server-integration-espi-adapter"
 				(path "/df391740-647e-4ab6-9dcd-d61184d66fe9/870b0b62-f962-4a87-8d30-5a8522c5db60"
-					(reference "R74")
+					(reference "R75")
 					(unit 1)
 				)
@@
 		(in_pos_files yes)
 		(dnp no)
-		(property "Reference" "R82"
+		(property "Reference" "R83"
 			(at 144.526 83.566 0)
 			(show_name no)
@@
 			(project "dc-scm-server-integration-espi-adapter"
 				(path "/df391740-647e-4ab6-9dcd-d61184d66fe9/870b0b62-f962-4a87-8d30-5a8522c5db60"
-					(reference "R82")
+					(reference "R83")
 					(unit 1)
 				)
@@
 		(in_pos_files yes)
 		(dnp no)
-		(property "Reference" "R78"
+		(property "Reference" "R79"
 			(at 144.526 73.406 0)
 			(show_name no)
@@
 			(project "dc-scm-server-integration-espi-adapter"
 				(path "/df391740-647e-4ab6-9dcd-d61184d66fe9/870b0b62-f962-4a87-8d30-5a8522c5db60"
-					(reference "R78")
+					(reference "R79")
 					(unit 1)
 				)
@@
 		(in_pos_files yes)
 		(dnp no)
-		(property "Reference" "#PWR091"
+		(property "Reference" "#PWR097"
 			(at 143.51 111.76 0)
 			(hide yes)
@@
 			(project "dc-scm-server-integration-espi-adapter"
 				(path "/df391740-647e-4ab6-9dcd-d61184d66fe9/870b0b62-f962-4a87-8d30-5a8522c5db60"
-					(reference "#PWR091")
+					(reference "#PWR097")
 					(unit 1)
 				)
@@
 		(dnp no)
 		(fields_autoplaced yes)
-		(property "Reference" "#PWR098"
+		(property "Reference" "#PWR0104"
 			(at 232.41 74.93 0)
 			(hide yes)
@@
 			(project "dc-scm-server-integration-espi-adapter"
 				(path "/df391740-647e-4ab6-9dcd-d61184d66fe9/870b0b62-f962-4a87-8d30-5a8522c5db60"
-					(reference "#PWR098")
+					(reference "#PWR0104")
 					(unit 1)
 				)
@@
 		(in_pos_files yes)
 		(dnp no)
-		(property "Reference" "#PWR092"
+		(property "Reference" "#PWR098"
 			(at 138.43 127 0)
 			(hide yes)
@@
 			(project "dc-scm-server-integration-espi-adapter"
 				(path "/df391740-647e-4ab6-9dcd-d61184d66fe9/870b0b62-f962-4a87-8d30-5a8522c5db60"
-					(reference "#PWR092")
+					(reference "#PWR098")
 					(unit 1)
 				)
@@
 		(in_pos_files yes)
 		(dnp no)
-		(property "Reference" "#PWR090"
+		(property "Reference" "#PWR096"
 			(at 104.14 55.88 0)
 			(hide yes)
@@
 			(project "dc-scm-server-integration-espi-adapter"
 				(path "/df391740-647e-4ab6-9dcd-d61184d66fe9/870b0b62-f962-4a87-8d30-5a8522c5db60"
-					(reference "#PWR090")
+					(reference "#PWR096")
 					(unit 1)
 				)
@@
 		(in_pos_files yes)
 		(dnp no)
-		(property "Reference" "R73"
+		(property "Reference" "R74"
 			(at 107.95 58.42 90)
 			(show_name no)
@@
 			(project "dc-scm-server-integration-espi-adapter"
 				(path "/df391740-647e-4ab6-9dcd-d61184d66fe9/870b0b62-f962-4a87-8d30-5a8522c5db60"
-					(reference "R73")
+					(reference "R74")
 					(unit 1)
 				)
@@
 		(in_pos_files yes)
 		(dnp no)
-		(property "Reference" "R79"
+		(property "Reference" "R80"
 			(at 144.526 75.946 0)
 			(show_name no)
@@
 			(project "dc-scm-server-integration-espi-adapter"
 				(path "/df391740-647e-4ab6-9dcd-d61184d66fe9/870b0b62-f962-4a87-8d30-5a8522c5db60"
-					(reference "R79")
+					(reference "R80")
 					(unit 1)
 				)
@@
 		(in_pos_files yes)
 		(dnp no)
-		(property "Reference" "R72"
+		(property "Reference" "R73"
 			(at 99.06 58.42 90)
 			(show_name no)
@@
 			(project "dc-scm-server-integration-espi-adapter"
 				(path "/df391740-647e-4ab6-9dcd-d61184d66fe9/870b0b62-f962-4a87-8d30-5a8522c5db60"
-					(reference "R72")
+					(reference "R73")
 					(unit 1)
 				)
@@
 		(in_pos_files yes)
 		(dnp no)
-		(property "Reference" "R71"
+		(property "Reference" "R72"
 			(at 90.17 58.42 90)
 			(show_name no)
@@
 			(project "dc-scm-server-integration-espi-adapter"
 				(path "/df391740-647e-4ab6-9dcd-d61184d66fe9/870b0b62-f962-4a87-8d30-5a8522c5db60"
-					(reference "R71")
+					(reference "R72")
 					(unit 1)
 				)
@@
 		(in_pos_files yes)
 		(dnp no)
-		(property "Reference" "R83"
+		(property "Reference" "R84"
 			(at 182.88 58.42 90)
 			(show_name no)
@@
 			(project "dc-scm-server-integration-espi-adapter"
 				(path "/df391740-647e-4ab6-9dcd-d61184d66fe9/870b0b62-f962-4a87-8d30-5a8522c5db60"
-					(reference "R83")
+					(reference "R84")
 					(unit 1)
 				)
@@
 		(in_pos_files yes)
 		(dnp no)
-		(property "Reference" "R76"
+		(property "Reference" "R77"
 			(at 134.62 58.42 90)
 			(show_name no)
@@
 			(project "dc-scm-server-integration-espi-adapter"
 				(path "/df391740-647e-4ab6-9dcd-d61184d66fe9/870b0b62-f962-4a87-8d30-5a8522c5db60"
-					(reference "R76")
+					(reference "R77")
 					(unit 1)
 				)
