File: port80-leds.kicad_sch (KiCad schematic)
At the start: 29 parts, among them U6001 SN74AC7541_VQFN, U6009 SN74AC7541_VQFN

Commit message: [#103753] Fixed issues according to the review
Connections:
- net +3V3: now also D6002.2 (A), D6003.2 (A), D6004.2 (A), D6005.2 (A), D6006.2 (A), D6007.2 (A), D6008.2 (A), D6009.2 (A)
- net 7SEG_L_A: now also D6008.1 (C)
- net 7SEG_L_A_R: no longer D6008.2 (A)
- net 7SEG_L_B: now also D6002.1 (C)
- net 7SEG_L_B_R: no longer D6002.2 (A)
- net 7SEG_L_C: now also D6003.1 (C)
- net 7SEG_L_C_R: no longer D6003.2 (A)
- net 7SEG_L_D: now also D6004.1 (C)
- net 7SEG_L_DP: now also D6009.1 (C)
- net 7SEG_L_DP_R: no longer D6009.2 (A)
- net 7SEG_L_D_R: no longer D6004.2 (A)
- net 7SEG_L_E: now also D6005.1 (C)
- net 7SEG_L_E_R: no longer D6005.2 (A)
- net 7SEG_L_F: now also D6006.1 (C)
- net 7SEG_L_F_R: no longer D6006.2 (A)
- net 7SEG_L_G: now also D6007.1 (C)
- net 7SEG_L_G_R: no longer D6007.2 (A)
- net GND: no longer D6002.1 (C), D6003.1 (C), D6004.1 (C), D6005.1 (C), D6006.1 (C), D6007.1 (C), D6008.1 (C), D6009.1 (C)
Other:
- moved on the sheet: D6002, D6003, D6004, D6005, D6006, D6007, D6008, D6009

Commit message: [#103697] Change redundant LED connections, start PCB layout
Connections:
- net 7SEG_L_A: no longer D6008.1 (C)
- net 7SEG_L_A_R: now also D6008.1 (C)
- net 7SEG_L_B: no longer D6002.1 (C)
- net 7SEG_L_B_R: now also D6002.1 (C)
- net 7SEG_L_C: no longer D6003.1 (C)
- net 7SEG_L_C_R: now also D6003.1 (C)
- net 7SEG_L_D: no longer D6004.1 (C)
- net 7SEG_L_DP: no longer D6009.1 (C)
- net 7SEG_L_DP_R: now also D6009.1 (C)
- net 7SEG_L_D_R: now also D6004.1 (C)
- net 7SEG_L_E: no longer D6005.1 (C)
- net 7SEG_L_E_R: now also D6005.1 (C)
- net 7SEG_L_F: no longer D6006.1 (C)
- net 7SEG_L_F_R: now also D6006.1 (C)
- net 7SEG_L_G: no longer D6007.1 (C)
- net 7SEG_L_G_R: now also D6007.1 (C)
Changed lines of the file:
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@@
-		)
-	)
-	(label "7SEG_L_A"
-		(at 151.13 115.57 0)
-		(effects
-			(font
-				(size 1.27 1.27)
-			)
-			(justify left bottom)
 		)
 	)
@@
 		)
 	)
-	(label "7SEG_L_G"
-		(at 151.13 146.05 0)
-		(effects
-			(font
-				(size 1.27 1.27)
-			)
-			(justify left bottom)
-		)
-	)
-	(label "7SEG_L_C"
-		(at 151.13 125.73 0)
-		(effects
-			(font
-				(size 1.27 1.27)
-			)
-			(justify left bottom)
-		)
-	)
 	(label "7SEG_L_C"
 		(at 200.66 87.63 0)
@@
 		)
 	)
-	(label "7SEG_L_F"
-		(at 151.13 140.97 0)
+	(label "7SEG_L_E_R"
+		(at 151.13 135.89 0)
+		(effects
+			(font
+				(size 1.27 1.27)
+			)
+			(justify left bottom)
+		)
+	)
+	(label "7SEG_L_D_R"
+		(at 151.13 130.81 0)
 		(effects
 			(font
@@
 		)
 	)
-	(label "7SEG_L_D"
-		(at 151.13 130.81 0)
-		(effects
-			(font
-				(size 1.27 1.27)
-			)
-			(justify left bottom)
-		)
-	)
 	(label "7SEG_H.G"
 		(at 45.72 97.79 0)
@@
 		)
 	)
-	(label "7SEG_L_DP"
-		(at 151.13 151.13 0)
-		(effects
-			(font
-				(size 1.27 1.27)
-			)
-			(justify left bottom)
-		)
-	)
 	(label "7SEG_H_F_R"
 		(at 111.76 95.25 0)
@@
 		)
 	)
+	(label "7SEG_L_F_R"
+		(at 151.13 140.97 0)
+		(effects
+			(font
+				(size 1.27 1.27)
+			)
+			(justify left bottom)
+		)
+	)
+	(label "7SEG_L_G_R"
+		(at 151.13 146.05 0)
+		(effects
+			(font
+				(size 1.27 1.27)
+			)
+			(justify left bottom)
+		)
+	)
 	(label "7SEG_H_G"
 		(at 77.47 97.79 0)
@@
 		)
 	)
-	(label "7SEG_L_E"
-		(at 151.13 135.89 0)
-		(effects
-			(font
-				(size 1.27 1.27)
-			)
-			(justify left bottom)
-		)
-	)
 	(label "7SEG_L.C"
 		(at 237.49 87.63 0)
@@
 		)
 	)
-	(label "7SEG_L_B"
-		(at 151.13 120.65 0)
-		(effects
-			(font
-				(size 1.27 1.27)
-			)
-			(justify left bottom)
-		)
-	)
 	(label "7SEG_L_D"
 		(at 200.66 90.17 0)
@@
 		)
 	)
+	(label "7SEG_L_DP_R"
+		(at 151.13 151.13 0)
+		(effects
+			(font
+				(size 1.27 1.27)
+			)
+			(justify left bottom)
+		)
+	)
 	(label "7SEG_L.D"
 		(at 237.49 90.17 0)
@@
 		(effects
 			(font
+				(size 1.27 1.27)
+			)
+			(justify left bottom)
+		)
+	)
+	(label "7SEG_L_C_R"
+		(at 151.13 125.73 0)
+		(effects
+			(font
+				(size 1.27 1.27)
+			)
+			(justify left bottom)
+		)
+	)
+	(label "7SEG_L_B_R"
+		(at 151.13 120.65 0)
+		(effects
+			(font
+				(size 1.27 1.27)
+			)
+			(justify left bottom)
+		)
+	)
+	(label "7SEG_L_A_R"
+		(at 151.13 115.57 0)
+		(effects
+			(font

Commit message: [#103697] Reenumerate the entire schematic, rerouting eSPI to maintain bigger gap between traces, rerouting the LDO
Parts:
- renumbered C6001 to C25, C6002 to C26, D6004 to D10, D6005 to D11, D6006 to D12, D6007 to D13, D6009 to D14, D6001 to D6, D6008 to D7, D6002 to D8, D6003 to D9, R6001 to R84, R6002 to R85, R6003 to R86, R6004 to R87, R6005 to R88, R6006 to R89, R6007 to R90, R6008 to R91, R6009 to R92, R6010 to R93, R6011 to R94, R6012 to R95, R6013 to R96, R6014 to R97, R6015 to R98, R6016 to R99, U6009 to U5, U6001 to U6

Commit message: [#103697] switch dc-dc for TPS566231PRQFR, eSPI length tuning, change zone clearance, fix clearance problems
Parts:
- renumbered C25 to C31, C26 to C32, R99 to R100, R84 to R85, R85 to R86, R86 to R87, R87 to R88, R88 to R89, R89 to R90, R90 to R91, R91 to R92, R92 to R93, R93 to R94, R94 to R95, R95 to R96, R96 to R97, R97 to R98, R98 to R99

Commit message: [#103697] pro: update name
Other:
- title: eSPI Adapter -> MEC1723 eSPI Debugger
Changed lines of the file:
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@@
 	(paper "A4")
 	(title_block
-		(title "eSPI Adapter")
-		(date "2026-08-21")
+		(title "MEC1723 eSPI Debugger")
+		(date "2026-09-02")
 		(rev "1.0.0")
 		(company "Antmicro")
@@
 		)
 		(instances
-			(project "dc-scm-server-integration-espi-adapter"
+			(project "mec1723-espi-debugger"
 				(path "/df391740-647e-4ab6-9dcd-d61184d66fe9/76679e57-0420-4874-b75d-368e938745be"
 					(reference "#PWR0105")
@@
 		)
 		(instances
-			(project "dc-scm-server-integration-espi-adapter"
+			(project "mec1723-espi-debugger"
 				(path "/df391740-647e-4ab6-9dcd-d61184d66fe9/76679e57-0420-4874-b75d-368e938745be"
 					(reference "D6")
@@
 		)
 		(instances
-			(project "dc-scm-server-integration-espi-adapter"
+			(project "mec1723-espi-debugger"
 				(path "/df391740-647e-4ab6-9dcd-d61184d66fe9/76679e57-0420-4874-b75d-368e938745be"
 					(reference "U6")
@@
 		)
 		(instances
-			(project "dc-scm-server-integration-espi-adapter"
+			(project "mec1723-espi-debugger"
 				(path "/df391740-647e-4ab6-9dcd-d61184d66fe9/76679e57-0420-4874-b75d-368e938745be"
 					(reference "R89")
@@
 		)
 		(instances
-			(project "dc-scm-server-integration-espi-adapter"
+			(project "mec1723-espi-debugger"
 				(path "/df391740-647e-4ab6-9dcd-d61184d66fe9/76679e57-0420-4874-b75d-368e938745be"
 					(reference "R88")
@@
 		)
 		(instances
-			(project "dc-scm-server-integration-espi-adapter"
+			(project "mec1723-espi-debugger"
 				(path "/df391740-647e-4ab6-9dcd-d61184d66fe9/76679e57-0420-4874-b75d-368e938745be"
 					(reference "R97")
@@
 		)
 		(instances
-			(project "dc-scm-server-integration-espi-adapter"
+			(project "mec1723-espi-debugger"
 				(path "/df391740-647e-4ab6-9dcd-d61184d66fe9/76679e57-0420-4874-b75d-368e938745be"
 					(reference "#PWR0109")
@@
 		)
 		(instances
-			(project "dc-scm-server-integration-espi-adapter"
+			(project "mec1723-espi-debugger"
 				(path "/df391740-647e-4ab6-9dcd-d61184d66fe9/76679e57-0420-4874-b75d-368e938745be"
 					(reference "R94")
@@
 		)
 		(instances
-			(project "dc-scm-server-integration-espi-adapter"
+			(project "mec1723-espi-debugger"
 				(path "/df391740-647e-4ab6-9dcd-d61184d66fe9/76679e57-0420-4874-b75d-368e938745be"
 					(reference "#PWR0112")
@@
 		)
 		(instances
-			(project "dc-scm-server-integration-espi-adapter"
+			(project "mec1723-espi-debugger"
 				(path "/df391740-647e-4ab6-9dcd-d61184d66fe9/76679e57-0420-4874-b75d-368e938745be"
 					(reference "U5")
@@
 		)
 		(instances
-			(project "dc-scm-server-integration-espi-adapter"
+			(project "mec1723-espi-debugger"
 				(path "/df391740-647e-4ab6-9dcd-d61184d66fe9/76679e57-0420-4874-b75d-368e938745be"
 					(reference "R85")
@@
 		)
 		(instances
-			(project "dc-scm-server-integration-espi-adapter"
+			(project "mec1723-espi-debugger"
 				(path "/df391740-647e-4ab6-9dcd-d61184d66fe9/76679e57-0420-4874-b75d-368e938745be"
 					(reference "R98")
@@
 		)
 		(instances
-			(project "dc-scm-server-integration-espi-adapter"
+			(project "mec1723-espi-debugger"
 				(path "/df391740-647e-4ab6-9dcd-d61184d66fe9/76679e57-0420-4874-b75d-368e938745be"
 					(reference "R87")
@@
 		)
 		(instances
-			(project "dc-scm-server-integration-espi-adapter"
+			(project "mec1723-espi-debugger"
 				(path "/df391740-647e-4ab6-9dcd-d61184d66fe9/76679e57-0420-4874-b75d-368e938745be"
 					(reference "#PWR0108")
@@
 		)
 		(instances
-			(project "dc-scm-server-integration-espi-adapter"
+			(project "mec1723-espi-debugger"
 				(path "/df391740-647e-4ab6-9dcd-d61184d66fe9/76679e57-0420-4874-b75d-368e938745be"
 					(reference "D11")
@@
 		)
 		(instances
-			(project "dc-scm-server-integration-espi-adapter"
+			(project "mec1723-espi-debugger"
 				(path "/df391740-647e-4ab6-9dcd-d61184d66fe9/76679e57-0420-4874-b75d-368e938745be"
 					(reference "R90")
@@
 		)
 		(instances
-			(project "dc-scm-server-integration-espi-adapter"
+			(project "mec1723-espi-debugger"
 				(path "/df391740-647e-4ab6-9dcd-d61184d66fe9/76679e57-0420-4874-b75d-368e938745be"
 					(reference "R86")
@@
 		)
 		(instances
-			(project "dc-scm-server-integration-espi-adapter"
+			(project "mec1723-espi-debugger"
 				(path "/df391740-647e-4ab6-9dcd-d61184d66fe9/76679e57-0420-4874-b75d-368e938745be"
 					(reference "R93")
@@
 		)
 		(instances
-			(project "dc-scm-server-integration-espi-adapter"
+			(project "mec1723-espi-debugger"
 				(path "/df391740-647e-4ab6-9dcd-d61184d66fe9/76679e57-0420-4874-b75d-368e938745be"
 					(reference "#PWR0106")
@@
 		)
 		(instances
-			(project "dc-scm-server-integration-espi-adapter"
+			(project "mec1723-espi-debugger"
 				(path "/df391740-647e-4ab6-9dcd-d61184d66fe9/76679e57-0420-4874-b75d-368e938745be"
 					(reference "#PWR0111")
@@
 		)
 		(instances
-			(project "dc-scm-server-integration-espi-adapter"
+			(project "mec1723-espi-debugger"
 				(path "/df391740-647e-4ab6-9dcd-d61184d66fe9/76679e57-0420-4874-b75d-368e938745be"
 					(reference "#PWR0107")
@@
 		)
 		(instances
-			(project "dc-scm-server-integration-espi-adapter"
+			(project "mec1723-espi-debugger"
 				(path "/df391740-647e-4ab6-9dcd-d61184d66fe9/76679e57-0420-4874-b75d-368e938745be"
 					(reference "D12")
@@
 		)
 		(instances
-			(project "dc-scm-server-integration-espi-adapter"
+			(project "mec1723-espi-debugger"
 				(path "/df391740-647e-4ab6-9dcd-d61184d66fe9/76679e57-0420-4874-b75d-368e938745be"
 					(reference "R95")
@@
 		)
 		(instances
-			(project "dc-scm-server-integration-espi-adapter"
+			(project "mec1723-espi-debugger"
 				(path "/df391740-647e-4ab6-9dcd-d61184d66fe9/76679e57-0420-4874-b75d-368e938745be"
 					(reference "#PWR0110")
@@
 		)
 		(instances
-			(project "dc-scm-server-integration-espi-adapter"
+			(project "mec1723-espi-debugger"
 				(path "/df391740-647e-4ab6-9dcd-d61184d66fe9/76679e57-0420-4874-b75d-368e938745be"
 					(reference "D9")
@@
 		)
 		(instances
-			(project "dc-scm-server-integration-espi-adapter"
+			(project "mec1723-espi-debugger"
 				(path "/df391740-647e-4ab6-9dcd-d61184d66fe9/76679e57-0420-4874-b75d-368e938745be"
 					(reference "#PWR0113")
@@
 		)
 		(instances
-			(project "dc-scm-server-integration-espi-adapter"
+			(project "mec1723-espi-debugger"
 				(path "/df391740-647e-4ab6-9dcd-d61184d66fe9/76679e57-0420-4874-b75d-368e938745be"
 					(reference "#PWR0115")
@@
 		)
 		(instances
-			(project "dc-scm-server-integration-espi-adapter"
+			(project "mec1723-espi-debugger"
 				(path "/df391740-647e-4ab6-9dcd-d61184d66fe9/76679e57-0420-4874-b75d-368e938745be"
 					(reference "D13")
@@
 		)
 		(instances
-			(project "dc-scm-server-integration-espi-adapter"
+			(project "mec1723-espi-debugger"
 				(path "/df391740-647e-4ab6-9dcd-d61184d66fe9/76679e57-0420-4874-b75d-368e938745be"
 					(reference "R91")
@@
 		)
 		(instances
-			(project "dc-scm-server-integration-espi-adapter"
+			(project "mec1723-espi-debugger"
 				(path "/df391740-647e-4ab6-9dcd-d61184d66fe9/76679e57-0420-4874-b75d-368e938745be"
 					(reference "R96")
@@
 		)
 		(instances
-			(project "dc-scm-server-integration-espi-adapter"
+			(project "mec1723-espi-debugger"
 				(path "/df391740-647e-4ab6-9dcd-d61184d66fe9/76679e57-0420-4874-b75d-368e938745be"
 					(reference "R99")
@@
 		)
 		(instances
-			(project "dc-scm-server-integration-espi-adapter"
+			(project "mec1723-espi-debugger"
 				(path "/df391740-647e-4ab6-9dcd-d61184d66fe9/76679e57-0420-4874-b75d-368e938745be"
 					(reference "D14")
@@
 		)
 		(instances
-			(project "dc-scm-server-integration-espi-adapter"
+			(project "mec1723-espi-debugger"
 				(path "/df391740-647e-4ab6-9dcd-d61184d66fe9/76679e57-0420-4874-b75d-368e938745be"
 					(reference "C31")
@@
 		)
 		(instances
-			(project "dc-scm-server-integration-espi-adapter"
+			(project "mec1723-espi-debugger"
 				(path "/df391740-647e-4ab6-9dcd-d61184d66fe9/76679e57-0420-4874-b75d-368e938745be"
 					(reference "D8")
@@
 		)
 		(instances
-			(project "dc-scm-server-integration-espi-adapter"
+			(project "mec1723-espi-debugger"
 				(path "/df391740-647e-4ab6-9dcd-d61184d66fe9/76679e57-0420-4874-b75d-368e938745be"
 					(reference "R92")
@@
 		)
 		(instances
-			(project "dc-scm-server-integration-espi-adapter"
+			(project "mec1723-espi-debugger"
 				(path "/df391740-647e-4ab6-9dcd-d61184d66fe9/76679e57-0420-4874-b75d-368e938745be"
 					(reference "D7")
@@
 		)
 		(instances
-			(project "dc-scm-server-integration-espi-adapter"
+			(project "mec1723-espi-debugger"
 				(path "/df391740-647e-4ab6-9dcd-d61184d66fe9/76679e57-0420-4874-b75d-368e938745be"
 					(reference "C32")
@@
 		)
 		(instances
-			(project "dc-scm-server-integration-espi-adapter"
+			(project "mec1723-espi-debugger"
 				(path "/df391740-647e-4ab6-9dcd-d61184d66fe9/76679e57-0420-4874-b75d-368e938745be"
 					(reference "R100")
@@
 		)
 		(instances
-			(project "dc-scm-server-integration-espi-adapter"
+			(project "mec1723-espi-debugger"
 				(path "/df391740-647e-4ab6-9dcd-d61184d66fe9/76679e57-0420-4874-b75d-368e938745be"
 					(reference "D10")
@@
 		)
 		(instances
-			(project "dc-scm-server-integration-espi-adapter"
+			(project "mec1723-espi-debugger"
 				(path "/df391740-647e-4ab6-9dcd-d61184d66fe9/76679e57-0420-4874-b75d-368e938745be"
 					(reference "#PWR0114")
