File: mec1723-espi-debugger.kicad_pcb (KiCad board)
At the start: 8 copper layers, 62 x 87 mm, 239 parts, among them J1 PinHeader_2x6_P2.54mm_Drill1.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, J10 PinHeader_2x5_P1.27mm_SMD, J11 PinHeader_2x5_P1.27mm_SMD, J12 PinHeader_2x5_P1.27mm_SMD, J13 Tag-Connect_TC2050-IDC-NL_2x5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, J14 Tag-Connect_TC2050-IDC-NL_2x5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, J15 USB-C_GCT_USB4105-GF-A, J2 PinHeader_2x5_P1.27mm_SMD, J3 PinHeader_2x5_P1.27mm_SMD, J4 PinHeader_2x5_P1.27mm_SMD, J5 PinHeader_2x5_P1.27mm_SMD, J6 PinHeader_2x5_P1.27mm_SMD, J7 PinHeader_2x5_P1.27mm_SMD, J8 PinHeader_2x5_P1.27mm_SMD, J9 PinHeader_2x5_P1.27mm_SMD, Q1 DMG1012T-7, SW1 SW_KSC441J70SHLFS_SMD, SW2 SW_KSC441J70SHLFS_SMD, SW3 SW_KSC441J70SHLFS_SMD, U1 MEC1723N-B0-I/SZ, U2 TLV76701_WSON, U3 TPS566231P, U4 MT25QU01GBBB8_SOIC, U5 SN74AC7541_VQFN, U6 SN74AC7541_VQFN, U7 FT2232HL-REEL, Y1 Resonator_32.768kHz_ECX-31B, Y2 Resonator_12MHz_KX-7

Commit message: [#103697] pcb: route VBUS on bottom and In6 layers
Routing:
- added copper zone on In6.Cu, net /Connectors/VBUS
Changed lines of the file:
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@@
 	(zone
 		(net "/Connectors/VBUS")
-		(layer "B.Cu")
+		(layers "B.Cu" "In6.Cu")
 		(hatch edge 0.5)
 		(priority 11)
